Commit message: message

File: rover_config/urdf/rover.urdf (robot description, URDF)
Before this commit: robot rover_model, 7 links, 6 joints
Links:
- added link arm2_connector2; visual cylinder length=0.1 radius=0.05
- added link arm2_link2; visual cylinder length=0.7 radius=0.05
- added link arm3_link3; visual cylinder length=0.4 radius=0.05
- added link arm_connector; visual cylinder length=0.1 radius=0.05
- added link arm_link; visual box size=0.1 0.1 1.0
- added link grip_connector; visual cylinder length=0.25 radius=0.05
- added link left_grip; visual cylinder length=0.25 radius=0.03
- added link right_grip; visual cylinder length=0.25 radius=0.03
- link base_link: geometry visual box size=0.7 1.4 0.4
Joints:
- added joint arm2_connector2_joint: type revolute, parent arm2_link2, child arm2_connector2, origin xyz=0 0.3 -0.1 rpy=0.0 0.0 0.0, axis 1 0 0, limit lower=0 upper=0 effort=0 velocity=0
- added joint arm2_link2_joint: type revolute, parent arm_connector, child arm2_link2, origin xyz=0 0.3 0 rpy=0.0 0.0 0.0, axis 1 0 0, limit lower=0 upper=0 effort=0 velocity=0
- added joint arm3_link3_joint: type revolute, parent arm2_connector2, child arm3_link3, origin xyz=0 0.05 -0.15 rpy=0.0 0.0 0.0, axis 1 0 0, limit lower=0 upper=0 effort=0 velocity=0
- added joint arm_connector_joint: type revolute, parent arm_link, child arm_connector, origin xyz=0 0 0.6 rpy=0.0 0.0 0.0, axis 1 0 0, limit lower=0 upper=0 effort=0 velocity=0
- added joint arm_link_joint: type revolute, parent base_link, child arm_link, origin xyz=0 0.45 0.4 rpy=0.0 0.0 0.0, axis 1 0 0, limit lower=0 upper=0 effort=0 velocity=0
- added joint grip_connector_joint: type revolute, parent arm3_link3, child grip_connector, origin xyz=0 0.1 -0.2 rpy=0.0 0.0 0.0, axis 1 0 0, limit lower=0 upper=0 effort=0 velocity=0
- added joint left_grip_joint: type revolute, parent grip_connector, child left_grip, origin xyz=0.07 0 -0.1 rpy=0.0 0.0 0.0, axis 1 0 0, limit lower=0 upper=0 effort=0 velocity=0
- added joint right_grip_joint: type revolute, parent grip_connector, child right_grip, origin xyz=-0.07 0 -0.1 rpy=0.0 0.0 0.0, axis 1 0 0, limit lower=0 upper=0 effort=0 velocity=0
- joint wheel_back_right_joint: origin xyz=-0.2 0.7 0.0 rpy=0.0 0.0 0.0 -> xyz=-0.2 0.7 0 rpy=0.0 0.0 0.0

Commit message: added inertia and collision models to some parts

File: rover_config/urdf/rover.urdf (robot description, URDF)
Before this commit: robot rover_model, 15 links, 14 joints
Links:
- link arm2_connector2: mass None -> 0.1
- link arm2_link2: mass None -> 0.1
- link arm3_link3: mass None -> 0.1
- link arm_connector: mass None -> 0.1
- link arm_link: mass None -> 0.1
- link base_link: mass None -> 30; geometry collision box size=0.7 1.4 0.4; visual box size=0.7 1.4 0.4
- link grip_connector: mass None -> 0.1
- link left_grip: mass None -> 0.1
- link left_rocker: mass None -> 1; geometry collision box size=0.2 1.4 0.2; visual box size=0.2 1.4 0.2
- link right_grip: mass None -> 0.1
- link right_rocker: mass None -> 1; geometry collision box size=0.2 1.4 0.2; visual box size=0.2 1.4 0.2
- link wheel_back_left: mass None -> 1; geometry collision cylinder length=0.2 radius=0.15; visual cylinder length=0.2 radius=0.15
- link wheel_back_right: mass None -> 1; geometry collision cylinder length=0.2 radius=0.15; visual cylinder length=0.2 radius=0.15
- link wheel_front_left: mass None -> 1; geometry collision cylinder length=0.2 radius=0.15; visual cylinder length=0.2 radius=0.15
- link wheel_front_right: mass None -> 1; geometry collision cylinder length=0.2 radius=0.15; visual cylinder length=0.2 radius=0.15
Joints:
- joint left_rocker_joint: limit lower=0.0 upper=0.0 effort=0.0 velocity=0.0 -> lower=-0.5235988 upper=0.5235988 effort=0.0 velocity=0.0
- joint right_rocker_joint: limit lower=0 upper=0 effort=0 velocity=0 -> lower=-0.5235988 upper=0.5235988 effort=0 velocity=0
- joint wheel_back_left_joint: limit lower=0 upper=0 effort=0 velocity=0 -> effort=0 velocity=0; type revolute -> continuous
- joint wheel_back_right_joint: limit lower=0 upper=0 effort=0 velocity=0 -> effort=0 velocity=0; type revolute -> continuous
- joint wheel_front_left_joint: limit lower=0 upper=0 effort=0 velocity=0 -> effort=0 velocity=0; type revolute -> continuous
- joint wheel_front_right_joint: limit lower=0 upper=0 effort=0 velocity=0 -> effort=0 velocity=0; type revolute -> continuous

Commit message: message

File: rover_config/urdf/rover.urdf (robot description, URDF)
Before this commit: robot rover_model, 15 links, 14 joints
Links:
- removed link arm2_connector2
- removed link arm_connector
Joints:
- removed joint arm2_connector2_joint
- removed joint arm_connector_joint
- joint arm2_link2_joint: origin xyz=0 0.3 0 rpy=0.0 0.0 0.0 -> xyz=0 0 0.70 rpy=0.0 0.0 0.0; parent arm_connector -> arm_link
- joint arm3_link3_joint: origin xyz=0 0.05 -0.15 rpy=0.0 0.0 0.0 -> xyz=0 -0.55 -0.13 rpy=0.0 0.0 0.0; parent arm2_connector2 -> arm2_link2
- joint arm_link_joint: origin xyz=0 0.45 0.4 rpy=0.0 0.0 0.0 -> xyz=0 -0.5 0.4 rpy=0.0 0.0 0.0
- joint grip_connector_joint: origin xyz=0 0.1 -0.2 rpy=0.0 0.0 0.0 -> xyz=0 -0.2 -0.3 rpy=0.0 0.0 0.0
- joint left_grip_joint: origin xyz=0.07 0 -0.1 rpy=0.0 0.0 0.0 -> xyz=0.07 -0.05 -0.1 rpy=0.0 0.0 0.0
- joint right_grip_joint: origin xyz=-0.07 0 -0.1 rpy=0.0 0.0 0.0 -> xyz=-0.07 -0.05 -0.1 rpy=0.0 0.0 0.0
