Commit message: fix the DiffDrive

File: rover_config/urdf/rover.urdf.xacro (robot description, xacro)
@@ -136,5 +136,5 @@
             <child link="wheel_${prefix}_${suffix}"/>
             <axis xyz="1 0 0"/>
-            <limit lower="0" upper="0" effort="0" velocity="0"/>
+            <!-- <limit lower="0" upper="0" effort="0" velocity="0"/> -->
         </joint>
         <gazebo reference="wheel_${prefix}_{suffix}_joint">

Commit message: Better skid steering

File: rover_config/urdf/rover.urdf.xacro (robot description, xacro)
@@ -1,4 +1,5 @@
 <?xml version="1.0"?>
-<robot name="rover_model" xmlns:xacro="http://www.ros.org/wiki/xacro">
+<robot name="rover_model"
+    xmlns:xacro="http://www.ros.org/wiki/xacro">
     <material name="black">
         <color rgba="0 0 0 1"/>
@@ -68,10 +69,11 @@
         <origin xyz="0.35 0.0 0.0" rpy="0.0 0.0 0.0"/>
         <axis xyz="1 0 0"/>
-        <limit lower="-0.5235988" upper="0.5235988" effort="0.0" velocity="0.0"/>
+        <!-- <limit lower="-0.5235988" upper="0.5235988" effort="0.0" velocity="0.0"/> -->
+        <limit lower="0" upper="0" effort="0.0" velocity="0.0"/>
     </joint>
     <transmission name="left_rocker_trans">
         <type>transmission_interface/SimpleTransmission</type>
         <joint name="left_rocker_joint">
-          <hardwareInterface>hardware_interface/EffortJointInterface</hardwareInterface>
+            <hardwareInterface>hardware_interface/EffortJointInterface</hardwareInterface>
         </joint>
         <actuator name="left_rocker_motor">
@@ -103,5 +105,6 @@
         <origin xyz="-0.35 0.0 0.0" rpy="0.0 0.0 0.0"/>
         <axis xyz="1 0 0"/>
-        <limit lower="-0.5235988" upper="0.5235988" effort="0" velocity="0"/>
+        <!-- <limit lower="-0.5235988" upper="0.5235988" effort="0" velocity="0"/> -->
+        <limit lower="0" upper="0" effort="0" velocity="0"/>
     </joint>
     <transmission name="right_rocker_trans">
@@ -139,8 +142,10 @@
         </joint>
         <gazebo reference="wheel_${prefix}_{suffix}_joint">
-            <mu1 value="2000.0"/>
-            <mu2 value="1000.0"/>
+            <!-- <mu1 value="200.0"/>
+            <mu2 value="100.0"/>
             <kp value="10000000.0" />
-            <kd value="1.0" />
+            <kd value="1.0" /> -->
+            <mu1>0.2</mu1>
+            <mu2>0.2</mu2>
             <material>Gazebo/Grey</material>
         </gazebo>
@@ -159,5 +164,5 @@
     <xacro:wheel prefix="back" suffix="left" reflect_x="1" reflect_y="-1"/>
     <xacro:wheel prefix="back" suffix="right" reflect_x="-1" reflect_y="-1"/>
-   <link name="arm_link">
+    <link name="arm_link">
         <visual>
             <geometry>
@@ -369,5 +374,5 @@
         <type>transmission_interface/SimpleTransmission</type>
         <joint name="arm_link_joint">
-          <hardwareInterface>hardware_interface/EffortJointInterface</hardwareInterface>
+            <hardwareInterface>hardware_interface/EffortJointInterface</hardwareInterface>
         </joint>
         <actuator name="arm_link_motor">
@@ -378,5 +383,5 @@
         <type>transmission_interface/SimpleTransmission</type>
         <joint name="arm_connector_joint">
-          <hardwareInterface>hardware_interface/EffortJointInterface</hardwareInterface>
+            <hardwareInterface>hardware_interface/EffortJointInterface</hardwareInterface>
         </joint>
         <actuator name="arm_connector_motor">
@@ -387,5 +392,5 @@
         <type>transmission_interface/SimpleTransmission</type>
         <joint name="arm2_link2_joint">
-          <hardwareInterface>hardware_interface/EffortJointInterface</hardwareInterface>
+            <hardwareInterface>hardware_interface/EffortJointInterface</hardwareInterface>
         </joint>
         <actuator name="arm2_link2_motor">
@@ -396,5 +401,5 @@
         <type>transmission_interface/SimpleTransmission</type>
         <joint name="arm2_connector2_joint">
-          <hardwareInterface>hardware_interface/EffortJointInterface</hardwareInterface>
+            <hardwareInterface>hardware_interface/EffortJointInterface</hardwareInterface>
         </joint>
         <actuator name="arm2_connector2_motor">
@@ -405,5 +410,5 @@
         <type>transmission_interface/SimpleTransmission</type>
         <joint name="arm3_link3_joint">
-          <hardwareInterface>hardware_interface/EffortJointInterface</hardwareInterface>
+            <hardwareInterface>hardware_interface/EffortJointInterface</hardwareInterface>
         </joint>
         <actuator name="arm3_link3_motor">
@@ -414,5 +419,5 @@
         <type>transmission_interface/SimpleTransmission</type>
         <joint name="grip_connector_joint">
-          <hardwareInterface>hardware_interface/EffortJointInterface</hardwareInterface>
+            <hardwareInterface>hardware_interface/EffortJointInterface</hardwareInterface>
         </joint>
         <actuator name="grip_connector_motor">
@@ -423,5 +428,5 @@
         <type>transmission_interface/SimpleTransmission</type>
         <joint name="left_grip_joint">
-          <hardwareInterface>hardware_interface/EffortJointInterface</hardwareInterface>
+            <hardwareInterface>hardware_interface/EffortJointInterface</hardwareInterface>
         </joint>
         <actuator name="left_grip_motor">
@@ -432,5 +437,5 @@
         <type>transmission_interface/SimpleTransmission</type>
         <joint name="right_grip_joint">
-          <hardwareInterface>hardware_interface/EffortJointInterface</hardwareInterface>
+            <hardwareInterface>hardware_interface/EffortJointInterface</hardwareInterface>
         </joint>
         <actuator name="right_grip_motor">
