Commit message: tune friction, remove rocker mimic

File: rover_config/urdf/test.xacro (robot description, xacro)
@@ -34,5 +34,5 @@
    <xacro:property name="rocker_width" value="0.1" />
    <!-- in meter -->
-   <xacro:property name="rocker_lenght" value="0.5" />
+   <xacro:property name="rocker_lenght" value="0.7" />
    <!-- in meter -->
    <xacro:property name="rocker_mass" value="2.0" />
@@ -116,5 +116,5 @@
          <mimic joint="right_rocker_joint" />
       </joint>
-      <transmission name="${side}_rocker_joint_trans" >
+      <!-- <transmission name="${side}_rocker_joint_trans" >
          <type>transmission_interface/SimpleTransmission</type>
          <joint name="${side}_rocker_joint">
@@ -123,9 +123,9 @@
          <actuator name="${side}_rocker_joint_motor">
             <hardwareInterface>hardware_interface/PositionJointInterface</hardwareInterface>
-            <mechanicalReduction>1</mechanicalReduction> <!-- It is not true: we uses motor with gearbox and ration of 75 -->
+            <mechanicalReduction>1</mechanicalReduction>
          </actuator>
-      </transmission>
-      <wheel fb="front" lr="${side}" parent="${side}_rocker" translateX="${rocker_lenght / 2}" translateY="${flipY * rocker_width}" translateZ="${-rocker_height / 2}" flipY="${flipY}"/>
-      <wheel fb="back" lr="${side}" parent="${side}_rocker" translateX="${-rocker_lenght / 2}" translateY="${flipY * rocker_width}" translateZ="${-rocker_height / 2}" flipY="${flipY}"/>
+      </transmission> -->
+      <wheel fb="front" lr="${side}" parent="${side}_rocker" translateX="${rocker_lenght / 2}" translateY="${flipY * rocker_width}" translateZ="${-rocker_height / 2}" flipY="${flipY}" flipZ="1"/>
+      <wheel fb="back" lr="${side}" parent="${side}_rocker" translateX="${-rocker_lenght / 2}" translateY="${flipY * rocker_width}" translateZ="${-rocker_height / 2}" flipY="${flipY}" flipZ="-1"/>
    </xacro:macro>
    <rocker side="left" parent="chassis" translateX="0" translateY="${base_width / 2}" translateZ="${-base_height / 2}" flipY="1" />
@@ -177,5 +177,5 @@
       </plugin>
    </gazebo>
-   <gazebo>
+   <!-- <gazebo>
       <plugin name="mimic_rocker" filename="libroboticsgroup_gazebo_mimic_joint_plugin.so">
          <joint>left_rocker_joint</joint>
@@ -185,4 +185,4 @@
          <hasPID/>
       </plugin>
-   </gazebo>
+   </gazebo> -->
 </robot>

File: rover_config/urdf/wheel.urdf.xacro (robot description, xacro)
@@ -10,5 +10,5 @@
                izz="${ m * r / 2}" />
    </xacro:macro>
-   <xacro:macro name="wheel" params="fb lr parent translateX translateY translateZ flipY">
+   <xacro:macro name="wheel" params="fb lr parent translateX translateY translateZ flipY flipZ">
    <!-- fb: front, back; lr: left right -->
       <link name="${fb}_${lr}_wheel">
@@ -34,8 +34,9 @@
       <gazebo reference="${fb}_${lr}_wheel" >
          <mu1 value="1.0"/>
-         <mu2 value="1.0" />
+         <!-- <mu2 value="1.0" /> -->
+         <mu2 value="0.1" />
          <kp  value="10000000.0" />
          <kd  value="1.0" />
-         <fdir1 value="1 1 0" />
+         <fdir1 value="1 ${flipY * flipZ} 0" />
          <slip1>0.5</slip1>
          <slip2>0</slip2>
