Commit message: fix arm limits

File: rover_config/urdf/arm.xacro (robot description, xacro)
@@ -1,4 +1,5 @@
 <?xml version="1.0" ?>
-<robot name="arm" xmlns:xacro="http://www.ros.org/wiki/xacro">
+<robot name="arm"
+    xmlns:xacro="http://www.ros.org/wiki/xacro">
     <xacro:property name="link0_len" value="0.01" />
     <xacro:property name="link0_rad" value="0.1" />
@@ -17,7 +18,13 @@
     <xacro:property name="offset_gripper" value="0.01" />
     <xacro:property name="lim_eff" value="30" />
-    <xacro:property name="lim_low" value="-2.617" />
-    <xacro:property name="lim_up" value="2.617" />
+    <xacro:property name="lim_low" value="-0.78539816339" />
+    <xacro:property name="lim_up" value="0.78539816339" />
     <xacro:property name="lim_vel" value="1.571" />
+    <xacro:macro name="box_inertia" params="m x y z">
+        <inertia ixx="${0.0833333 * m * (y*y + z*z)}" ixy="0.0" ixz="0.0" iyy="${0.0833333 * m * (x*x + z*z)}" iyz="0.0" izz="${0.0833333 * m * (x*x + y*y)}" />
+    </xacro:macro>
+    <xacro:macro name="cylinder_inertia" params="m r h">
+        <inertia ixx="${ m * ( 3 * r*r + h*h ) / 12}" ixy="0" ixz="0" iyy="${ m * ( 3 * r*r + h*h ) / 12}" iyz="0" izz="${ m * r / 2}" />
+    </xacro:macro>
     <material name="black">
         <color rgba="0.0 0.0 0.0 1.0"/>
@@ -30,7 +37,7 @@
             <parent link="${parent}"/>
             <child link="link0"/>
-            <origin rpy="0 0 0" xyz="${-translateX} ${-translateY} ${-translateZ}"/>
+            <origin rpy="0 0 0" xyz="${translateX} ${translateY} ${translateZ}"/>
             <axis xyz="0 0 1"/>
-            <limit effort="${lim_eff}" lower="${lim_low}" upper="${lim_low}" velocity="${lim_vel}"/>
+            <limit effort="${lim_eff}" lower="${lim_low}" upper="${lim_up}" velocity="${lim_vel}"/>
         </joint>
         <link name="link0">
@@ -51,14 +58,13 @@
                 <origin rpy="0 0 0" xyz="0 0 ${link0_len/2}"/>
                 <mass value="1"/>
-                <inertia ixx="1.0" ixy="0.0" ixz="0.0" iyy="1.0" iyz="0.0" izz="1.0"/>
-            </inertial>
-        </link>
-<!--
+                <cylinder_inertia m="1" r="${link0_rad}" h="${link0_len}" />
+            </inertial>
+        </link>
         <joint name="joint0" type="revolute">
             <parent link="link0"/>
             <child link="link1"/>
-            <origin rpy="0 0 0" xyz="0 0 ${-link0_len}"/>
+            <origin rpy="0 0 0" xyz="0 0 ${link0_len}"/>
             <axis xyz="0 1 0"/>
-            <limit effort="${lim_eff}" lower="${lim_low}" upper="${lim_low}" velocity="${lim_vel}"/>
+            <limit effort="${lim_eff}" lower="${lim_low}" upper="${lim_up}" velocity="${lim_vel}"/>
         </joint>
         <link name="link1">
@@ -72,5 +78,5 @@
                 <origin rpy="0 0 0" xyz="0 0 ${link1_len/2}"/>
                 <geometry>
-                <box size="${link1_width} ${link1_width} ${link1_len}"/>
+                    <box size="${link1_width} ${link1_width} ${link1_len}"/>
                 </geometry>
                 <material name="black"/>
@@ -79,5 +85,5 @@
                 <origin rpy="0 0 0" xyz="0 0 ${link1_len/2}"/>
                 <mass value="1"/>
-                <inertia ixx="1.0" ixy="0.0" ixz="0.0" iyy="1.0" iyz="0.0" izz="1.0"/>
+                <box_inertia m="1" x="${link1_width}" y="${link1_width}" z="${link1_len}" />
             </inertial>
         </link>
@@ -85,7 +91,7 @@
             <parent link="link1"/>
             <child link="link2"/>
-            <origin rpy="0 0 0" xyz="0 0 ${-link1_len}"/>
+            <origin rpy="0 0 0" xyz="0 0 ${link1_len}"/>
             <axis xyz="0 1 0"/>
-            <limit effort="${lim_eff}" lower="${lim_low}" upper="${lim_low}" velocity="${lim_vel}"/>
+            <limit effort="${lim_eff}" lower="${lim_low}" upper="${lim_up}" velocity="${lim_vel}"/>
         </joint>
         <link name="link2">
@@ -93,5 +99,5 @@
                 <origin rpy="0 0 0" xyz="0 0 ${link2_len/2}"/>
                 <geometry>
-                <box size="${link2_width} ${link2_width} ${link2_len}"/>
+                    <box size="${link2_width} ${link2_width} ${link2_len}"/>
                 </geometry>
             </collision>
@@ -99,12 +105,12 @@
                 <origin rpy="0 0 0" xyz="0 0 ${link2_len/2}"/>
                 <geometry>
-                <box size="${link2_width} ${link2_width} ${link2_len}"/>
+                    <box size="${link2_width} ${link2_width} ${link2_len}"/>
                 </geometry>
                 <material name="orange"/>
             </visual>
-                <inertial>
+            <inertial>
                 <origin rpy="0 0 0" xyz="0 0 ${link2_len/2}"/>
                 <mass value="1"/>
-                <inertia ixx="1.0" ixy="0.0" ixz="0.0" iyy="1.0" iyz="0.0" izz="1.0"/>
+                <box_inertia m="1" x="${link2_width}" y="${link2_width}" z="${link2_len}" />
             </inertial>
         </link>
@@ -112,7 +118,7 @@
             <parent link="link2"/>
             <child link="link3"/>
-            <origin rpy="0 0 0" xyz="0 0 ${-link2_len}"/>
+            <origin rpy="0 0 0" xyz="0 0 ${link2_len}"/>
             <axis xyz="0 0 1"/>
-            <limit effort="${lim_eff}" lower="${lim_low}" upper="${lim_low}" velocity="${lim_vel}"/>
+            <limit effort="${lim_eff}" lower="${lim_low}" upper="${lim_up}" velocity="${lim_vel}"/>
         </joint>
         <link name="link3">
@@ -120,5 +126,5 @@
                 <origin rpy="0 0 0" xyz="0 0 ${link3_len/2}"/>
                 <geometry>
-                <box size="${link3_width} ${link3_width} ${link3_len}"/>
+                    <box size="${link3_width} ${link3_width} ${link3_len}"/>
                 </geometry>
             </collision>
@@ -126,5 +132,5 @@
                 <origin rpy="0 0 0" xyz="0 0 ${link3_len/2}"/>
                 <geometry>
-                <box size="${link3_width} ${link3_width} ${link3_len}"/>
+                    <box size="${link3_width} ${link3_width} ${link3_len}"/>
                 </geometry>
                 <material name="black"/>
@@ -133,5 +139,5 @@
                 <origin rpy="0 0 0" xyz="0 0 ${link3_len/2}"/>
                 <mass value="1"/>
-                <inertia ixx="1.0" ixy="0.0" ixz="0.0" iyy="1.0" iyz="0.0" izz="1.0"/>
+                <box_inertia m="1" x="${link3_width}" y="${link3_width}" z="${link3_len}" />
             </inertial>
         </link>
@@ -139,7 +145,7 @@
             <parent link="link3"/>
             <child link="link4"/>
-            <origin rpy="0 0 0" xyz="0 0 ${-link3_len}"/>
+            <origin rpy="0 0 0" xyz="0 0 ${link3_len}"/>
             <axis xyz="0 1 0"/>
-            <limit effort="${lim_eff}" lower="${lim_low}" upper="${lim_low}" velocity="${lim_vel}"/>
+            <limit effort="${lim_eff}" lower="${lim_low}" upper="${lim_up}" velocity="${lim_vel}"/>
         </joint>
         <link name="link4">
@@ -147,5 +153,5 @@
                 <origin rpy="0 0 0" xyz="0 0 ${link4_len/2}"/>
                 <geometry>
-                <box size="${link4_width} ${link4_width} ${link4_len}"/>
+                    <box size="${link4_width} ${link4_width} ${link4_len}"/>
                 </geometry>
             </collision>
@@ -153,5 +159,5 @@
                 <origin rpy="0 0 0" xyz="0 0 ${link4_len/2}"/>
                 <geometry>
-                <box size="${link4_width} ${link4_width} ${link4_len}"/>
+                    <box size="${link4_width} ${link4_width} ${link4_len}"/>
                 </geometry>
                 <material name="orange"/>
@@ -160,5 +166,5 @@
                 <origin rpy="0 0 0" xyz="0 0 ${link4_len/2}"/>
                 <mass value="1"/>
-                <inertia ixx="1.0" ixy="0.0" ixz="0.0" iyy="1.0" iyz="0.0" izz="1.0"/>
+                <box_inertia m="1" x="${link4_width}" y="${link4_width}" z="${link4_len}" />
             </inertial>
         </link>
@@ -166,7 +172,7 @@
             <parent link="link4"/>
             <child link="link5"/>
-            <origin rpy="0 0 0" xyz="0 0 ${-link4_len}"/>
+            <origin rpy="0 0 0" xyz="0 0 ${link4_len}"/>
             <axis xyz="0 0 1"/>
-            <limit effort="${lim_eff}" lower="${lim_low}" upper="${lim_low}" velocity="${lim_vel}"/>
+            <limit effort="${lim_eff}" lower="${lim_low}" upper="${lim_up}" velocity="${lim_vel}"/>
         </joint>
         <link name="link5">
@@ -174,5 +180,5 @@
                 <origin rpy="0 0 0" xyz="0 0 ${link5_len/2}"/>
                 <geometry>
-                <box size="${link5_width} ${link5_width} ${link5_len}"/>
+                    <box size="${link5_width} ${link5_width} ${link5_len}"/>
                 </geometry>
             </collision>
@@ -180,5 +186,5 @@
                 <origin rpy="0 0 0" xyz="0 0 ${link5_len/2}"/>
                 <geometry>
-                <box size="${link5_width} ${link5_width} ${link5_len}"/>
+                    <box size="${link5_width} ${link5_width} ${link5_len}"/>
                 </geometry>
                 <material name="black"/>
@@ -187,5 +193,5 @@
                 <origin rpy="0 0 0" xyz="0 0 ${link5_len/2}"/>
                 <mass value="1"/>
-                <inertia ixx="1.0" ixy="0.0" ixz="0.0" iyy="1.0" iyz="0.0" izz="1.0"/>
+                <box_inertia m="1" x="${link5_width}" y="${link5_width}" z="${link5_len}" />
             </inertial>
         </link>
@@ -193,14 +199,14 @@
             <parent link="link5"/>
             <child link="gripper_left"/>
-            <origin rpy="0 0 0" xyz="0 ${offset_gripper} ${-link5_len}"/>
+            <origin rpy="0 0 0" xyz="0 ${offset_gripper} ${link5_len}"/>
             <axis xyz="1 0 0"/>
-            <limit effort="${lim_eff}" lower="${lim_low}" upper="${lim_low}" velocity="${lim_vel}"/>
+            <limit effort="${lim_eff}" lower="${lim_low}" upper="${lim_up}" velocity="${lim_vel}"/>
         </joint>
         <joint name="joint6" type="revolute">
             <parent link="link5"/>
             <child link="gripper_right"/>
-            <origin rpy="0 0 0" xyz="0 -${offset_gripper} ${-link5_len}"/>
+            <origin rpy="0 0 0" xyz="0 -${offset_gripper} ${link5_len}"/>
             <axis xyz="1 0 0"/>
-            <limit effort="${lim_eff}" lower="${lim_low}" upper="${lim_low}" velocity="${lim_vel}"/>
+            <limit effort="${lim_eff}" lower="${lim_low}" upper="${lim_up}" velocity="${lim_vel}"/>
         </joint>
         <link name="gripper_left">
@@ -221,5 +227,5 @@
                 <origin rpy="0 0 0" xyz="0 0 ${gripper_len/2}"/>
                 <mass value="1"/>
-                <inertia ixx="1.0" ixy="0.0" ixz="0.0" iyy="1.0" iyz="0.0" izz="1.0"/>
+                <cylinder_inertia m="1" r="${gripper_rad}" h="${gripper_len}" />
             </inertial>
         </link>
@@ -241,10 +247,9 @@
                 <origin rpy="0 0 0" xyz="0 0 ${gripper_len/2}"/>
                 <mass value="1"/>
-                <inertia ixx="1.0" ixy="0.0" ixz="0.0" iyy="1.0" iyz="0.0" izz="1.0"/>
-            </inertial>
-        </link>
--->
+                <cylinder_inertia m="1" r="${gripper_rad}" h="${gripper_len}" />
+            </inertial>
+        </link>
         <!-- Transmission is important to link the joint and the controller -->
-<!--
+        <!--
         <transmission name="joint_base_trans">
             <type>transmission_interface/SimpleTransmission</type>
@@ -319,5 +324,5 @@
             </actuator>
         </transmission>
--->
+        -->
     </xacro:macro>
 </robot>

File: rover_config/urdf/testarm.xacro (robot description, xacro)
@@ -4,5 +4,5 @@
       <link name="base_link">
         <collision>
-          <origin rpy="0 0 0" xyz="0.0 0.0 0.1"/>
+          <origin rpy="0 0 0" xyz="0.0 0.0 0.0"/>
           <geometry>
             <cylinder length="0.1" radius="0.5"/>
@@ -10,5 +10,5 @@
         </collision>
         <visual>
-          <origin rpy="0 0 0" xyz="0.0 0.0 0.1"/>
+          <origin rpy="0 0 0" xyz="0.0 0.0 0.0"/>
           <geometry>
             <cylinder length="0.1" radius="0.5"/>
@@ -17,15 +17,14 @@
         <inertial>
             <origin rpy="0 0 0" xyz="0 0 0"/>
-            <mass value="1"/>
-            <inertia ixx="1.0" ixy="0.0" ixz="0.0" iyy="1.0" iyz="0.0" izz="1.0"/>
+            <mass value="100"/>
+            <cylinder_inertia m="100" r="${0.5}" h="${0.1}" />
         </inertial>
       </link>
-      <arm parent="base_link" translateX="0.3" translateY="0.2" translateZ="0.1"/>
-<!--
+      <arm parent="base_link" translateX="0.3" translateY="0" translateZ="0.05"/>
    <gazebo>
       <plugin name="joint_state_publisher" filename="libgazebo_ros_joint_state_publisher.so">
          <jointName>
-            joint01,
-            joint02,
+            joint_base,
+            joint0,
             joint1,
             joint2,
@@ -40,6 +39,5 @@
       </plugin>
    </gazebo>
--->
-   <gazebo>
+   <!-- <gazebo>
       <plugin name="gazebo_ros_control" filename="libgazebo_ros_control.so">
          <robotNamespace>/</robotNamespace>
@@ -47,4 +45,4 @@
          <legacyModeNS>true</legacyModeNS>
       </plugin>
-   </gazebo>
+   </gazebo> -->
 </robot>

Commit message: motor joints can be controlled with rostopic pub

File: rover_config/urdf/arm.xacro (robot description, xacro)
@@ -17,5 +17,5 @@
     <xacro:property name="gripper_rad" value="0.01" />
     <xacro:property name="offset_gripper" value="0.01" />
-    <xacro:property name="lim_eff" value="30" />
+    <xacro:property name="lim_eff" value="300" />
     <xacro:property name="lim_low" value="-0.78539816339" />
     <xacro:property name="lim_up" value="0.78539816339" />
@@ -251,5 +251,4 @@
         </link>
         <!-- Transmission is important to link the joint and the controller -->
-        <!--
         <transmission name="joint_base_trans">
             <type>transmission_interface/SimpleTransmission</type>
@@ -323,6 +322,5 @@
                 <mechanicalReduction>1</mechanicalReduction>
             </actuator>
-        </transmission>
-        -->
+            </transmission>
     </xacro:macro>
 </robot>

File: rover_config/urdf/testarm.xacro (robot description, xacro)
@@ -46,3 +46,8 @@
       </plugin>
    </gazebo> -->
+    <gazebo>
+        <plugin name="gazebo_ros_control" filename="libgazebo_ros_control.so">
+            <robotNamespace>/nimrod</robotNamespace>
+        </plugin>
+    </gazebo>
 </robot>

Commit message: testing, structure is not nice, MoveIt setup assistant package

File: rover_config/urdf/arm.xacro (robot description, xacro)
@@ -2,5 +2,5 @@
 <robot name="arm"
     xmlns:xacro="http://www.ros.org/wiki/xacro">
-    <xacro:property name="link0_len" value="0.01" />
+    <xacro:property name="link0_len" value="0.1" />
     <xacro:property name="link0_rad" value="0.1" />
     <xacro:property name="link1_len" value="0.6" />
@@ -18,6 +18,6 @@
     <xacro:property name="offset_gripper" value="0.01" />
     <xacro:property name="lim_eff" value="300" />
-    <xacro:property name="lim_low" value="-0.78539816339" />
-    <xacro:property name="lim_up" value="0.78539816339" />
+    <xacro:property name="lim_low" value="-1.78539816339" />
+    <xacro:property name="lim_up" value="1.78539816339" />
     <xacro:property name="lim_vel" value="1.571" />
     <xacro:macro name="box_inertia" params="m x y z">
@@ -53,5 +53,5 @@
                     <cylinder length="${link0_len}" radius="${link0_rad}"/>
                 </geometry>
-                <material name="black"/>
+                <material name="orange"/>
             </visual>
             <inertial>
