Commit message: fix rotation issue and stabelize the body

File: rover_config/urdf/rover.xacro (robot description, xacro)
@@ -23,19 +23,12 @@
    <!-- Main body length height width -->
    <xacro:property name="base_height" value="0.2" />
-   <!-- in meter -->
    <xacro:property name="base_width" value="0.2" />
-   <!-- in meter -->
    <xacro:property name="base_lenght" value="0.5" />
-   <!-- in meter -->
    <xacro:property name="base_mass" value="20.0" />
-   <!-- in kg -->
    <xacro:property name="rocker_height" value="0.1" />
-   <!-- in meter -->
    <xacro:property name="rocker_width" value="0.1" />
-   <!-- in meter -->
    <xacro:property name="rocker_lenght" value="0.7" />
-   <!-- in meter -->
    <xacro:property name="rocker_mass" value="2.0" />
-   <!-- in kg -->
+   <xacro:property name="rocker_offsetZ" value="0.2" />
    <!-- Macro for calculating inertia of cylinder -->
    <xacro:macro name="cylinder_inertia" params="m r h">
@@ -50,5 +43,5 @@
    <!-- It is necessary as gazebo does not support inertia for the root link -->
    <!-- Do not call it world as it is reserved for robot that must be fixed to the world -->
-   <link name="base_link">
+  <link name="base_link">
    </link>
    <gazebo reference="base_link">
@@ -90,5 +83,5 @@
       <link name="${side}_rocker">
          <visual>
-            <origin xyz="0 ${flipY * rocker_width / 2} 0" rpy="0 0 0"/>
+            <origin xyz="0 ${flipY * rocker_width / 2} ${-rocker_offsetZ}" rpy="0 0 0"/>
             <geometry>
                <box size="${rocker_lenght} ${rocker_width} ${rocker_height}" />
@@ -97,5 +90,5 @@
          </visual>
          <collision>
-            <origin xyz="0 ${flipY * rocker_width / 2} 0" rpy="0 0 0"/>
+            <origin xyz="0 ${flipY * rocker_width / 2} ${-rocker_offsetZ}" rpy="0 0 0"/>
             <geometry>
                <box size="${rocker_lenght} ${rocker_width} ${rocker_height}" />
@@ -104,5 +97,5 @@
          <inertial>
             <mass value="${rocker_mass}" />
-            <origin xyz="0 0 0" />
+            <origin xyz="0 ${flipY * rocker_width / 2} ${-rocker_offsetZ}" rpy="0 0 0"/>
             <box_inertia m="${rocker_mass}" x="${rocker_lenght}" y="${rocker_width}" z="${rocker_height}" />
          </inertial>
@@ -113,8 +106,8 @@
          <child link="${side}_rocker"/>
          <axis xyz="0 1 0"/>
-         <limit lower="${-30 * DEG_TO_RAD}" upper="${30 * DEG_TO_RAD}" effort="10000.0" velocity="100000.0"/>
-         <mimic joint="right_rocker_joint" />
+         <dynamics damping="0" friction="0.5"/>
+         <limit lower="${-30 * DEG_TO_RAD}" upper="${30 * DEG_TO_RAD}" velocity="1000" effort="1000"/>
       </joint>
-      <!-- <transmission name="${side}_rocker_joint_trans" >
+      <transmission name="${side}_rocker_joint_trans">
          <type>transmission_interface/SimpleTransmission</type>
          <joint name="${side}_rocker_joint">
@@ -125,10 +118,10 @@
             <mechanicalReduction>1</mechanicalReduction>
          </actuator>
-      </transmission> -->
-      <wheel fb="front" lr="${side}" parent="${side}_rocker" translateX="${rocker_lenght / 2}" translateY="${flipY * rocker_width}" translateZ="${-rocker_height / 2}" flipY="${flipY}" flipZ="1"/>
-      <wheel fb="back" lr="${side}" parent="${side}_rocker" translateX="${-rocker_lenght / 2}" translateY="${flipY * rocker_width}" translateZ="${-rocker_height / 2}" flipY="${flipY}" flipZ="-1"/>
+      </transmission>
+      <wheel fb="front" lr="${side}" parent="${side}_rocker" translateX="${rocker_lenght / 2}" translateY="${flipY * rocker_width}" translateZ="${-rocker_offsetZ -rocker_height / 2}" flipY="${flipY}" flipZ="1"/>
+      <wheel fb="back" lr="${side}" parent="${side}_rocker" translateX="${-rocker_lenght / 2}" translateY="${flipY * rocker_width}" translateZ="${-rocker_offsetZ -rocker_height / 2}" flipY="${flipY}" flipZ="-1"/>
    </xacro:macro>
-   <rocker side="left" parent="chassis" translateX="0" translateY="${base_width / 2}" translateZ="${-base_height / 2}" flipY="1" />
-   <rocker side="right" parent="chassis" translateX="0" translateY="${-base_width / 2}" translateZ="${-base_height / 2}" flipY="-1" />
+   <rocker side="left" parent="chassis" translateX="0" translateY="${base_width / 2}" translateZ="${-base_height / 3}" flipY="1" />
+   <rocker side="right" parent="chassis" translateX="0" translateY="${-base_width / 2}" translateZ="${-base_height / 3}" flipY="-1" />
    <!-- Wheel Definition for simulation -->
    <!-- <wheel fb="front" lr="right" parent="chassis" translateX="0.4" translateY="${-1*(base_width/2+0.04)}" translateZ="-0.065" flipY="1"/>
@@ -137,5 +130,5 @@
    <wheel fb="back" lr="left" parent="chassis" translateX="-0.4" translateY="${1*(base_width/2+0.04)}" translateZ="-0.065" flipY="1"/> -->
    <!-- Skid Steering Drive for 4 wheel robot for simulation -->
-   <gazebo>
+   <!-- <gazebo>
       <plugin name="drive_controller" filename="libgazebo_ros_skid_steer_drive.so">
          <updateRate>100</updateRate>
@@ -158,5 +151,5 @@
          <covariance_yaw>0.010000</covariance_yaw>
       </plugin>
-   </gazebo>
+   </gazebo> -->
    <!-- Publishing joint states from Gazebo simulator -->
    <!-- fixed links are not published -->
@@ -177,12 +170,16 @@
       </plugin>
    </gazebo>
-   <!-- <gazebo>
+   <gazebo>
+      <plugin name="gazebo_ros_control" filename="libgazebo_ros_control.so">
+         <robotNamespace>/</robotNamespace>
+      </plugin>
+   </gazebo>
+   <gazebo>
       <plugin name="mimic_rocker" filename="libroboticsgroup_gazebo_mimic_joint_plugin.so">
          <joint>left_rocker_joint</joint>
-         <mimicJoint>right_rocker</mimicJoint>
+         <mimicJoint>right_rocker_joint</mimicJoint>
          <multiplier>-1</multiplier>
-         <maxEffort>1000</maxEffort>
-         <hasPID/>
+         <hasPID />
       </plugin>
-   </gazebo> -->
+   </gazebo>
 </robot>

File: rover_config/urdf/wheel.urdf.xacro (robot description, xacro)
@@ -1,18 +1,61 @@
 <?xml version="1.0"?>
-<robot name="wheel" xmlns:xacro="http://www.ros.org/wiki/xacro">
-<xacro:property name="wheel_radius" value="0.15" />
-<xacro:property name="wheel_width"  value="0.2"  />
-<xacro:property name="wheel_mass"   value="1"  />  <!-- in kg -->
+<robot name="wheel"
+   xmlns:xacro="http://www.ros.org/wiki/xacro">
+   <xacro:property name="wheel_radius" value="0.15" />
+   <xacro:property name="wheel_width" value="0.2" />
+   <xacro:property name="wheel_mass" value="1" />
+   <!-- in kg -->
    <!-- Macro for calculating inertia of cylindric wheel -->
    <xacro:macro name="wheel_inertia" params="m r h">
-      <inertia ixx="${ m * ( 3 * r*r + h*h ) / 12}" ixy="0" ixz="0"
-               iyy="${ m * ( 3 * r*r + h*h ) / 12}" iyz="0"
-               izz="${ m * r / 2}" />
+      <inertia ixx="${ m * ( 3 * r*r + h*h ) / 12}" ixy="0" ixz="0" iyy="${ m * ( 3 * r*r + h*h ) / 12}" iyz="0" izz="${ m * r / 2}" />
+   </xacro:macro>
+   <xacro:macro name="grouser" params="links_qty max_qty parent flipY flipZ">
+      <link name="${flipY}${flipZ}_${links_qty}">
+         <visual>
+            <origin xyz="0 ${flipY * wheel_width / 2} ${wheel_radius}" rpy="0 0 ${flipY * flipZ * 30 * DEG_TO_RAD}"/>
+            <geometry>
+               <box size="0.01 ${wheel_width} 0.05"/>
+            </geometry>
+            <material name="Red" />
+         </visual>
+         <collision>
+            <origin xyz="0 ${flipY * wheel_width / 2} ${wheel_radius}" rpy="0 0 ${flipY * flipZ * 30 * DEG_TO_RAD}"/>
+            <geometry>
+               <box size="0.01 ${wheel_width} 0.05"/>
+            </geometry>
+            <material name="Red" />
+         </collision>
+         <inertial>
+            <mass value="0.01" />
+            <origin xyz="0 ${flipY * wheel_width / 2} ${wheel_radius}" rpy="0 0 ${flipY * flipZ * 30 * DEG_TO_RAD}"/>
+            <box_inertia m="0.01" x="0.01" y="${wheel_width}" z="0.05" />
+         </inertial>
+      </link>
+      <joint name="${flipY}${flipZ}_${links_qty}_joint" type="fixed">
+         <parent link="${parent}"/>
+         <child link="${flipY}${flipZ}_${links_qty}" />
+         <origin xyz="0.0 0.0 0.0" rpy="0 ${links_qty * 360 / max_qty * DEG_TO_RAD} 0" />
+      </joint>
+      <gazebo reference="${flipY}${flipZ}_${links_qty}">
+         <mu1 value="10"/>
+         <mu2 value="0.1" />
+         <!-- <mu2 value="1" /> -->
+         <!-- <fdir1 value="0.7071 ${-flipY * flipZ * 0.7071} 0" /> -->
+         <fdir1 value="1 0 0" />
+         <kp value="10000000.0" />
+         <kd value="1.0" />
+         <material>Gazebo/Black</material>
+         <turnGravityOff>false</turnGravityOff>
+      </gazebo>
+      <xacro:if value="${links_qty}">
+         <xacro:grouser links_qty="${links_qty - 1}" max_qty="${max_qty}" parent="${parent}" flipY="${flipY}" flipZ="${flipZ}" />
+      </xacro:if>
    </xacro:macro>
    <xacro:macro name="wheel" params="fb lr parent translateX translateY translateZ flipY flipZ">
-   <!-- fb: front, back; lr: left right -->
+      <!-- fb: front, back; lr: left right -->
       <link name="${fb}_${lr}_wheel">
          <visual>
-            <origin xyz="0 ${flipY * wheel_width / 2} 0" rpy="${flipY*M_PI/2} 0 0"/>  <!-- make sure the wheel is in the correct position -->
+            <origin xyz="0 ${flipY * wheel_width / 2} 0" rpy="${flipY*M_PI/2} 0 0"/>
+            <!-- make sure the wheel is in the correct position -->
             <geometry>
                <cylinder length="${wheel_width}" radius="${wheel_radius}" />
@@ -32,14 +75,6 @@
          </inertial>
       </link>
-      <gazebo reference="${fb}_${lr}_wheel" >
-         <mu1 value="1.0"/>
-         <!-- <mu2 value="1.0" /> -->
-         <mu2 value="0.1" />
-         <kp  value="10000000.0" />
-         <kd  value="1.0" />
-         <fdir1 value="1 ${flipY * flipZ} 0" />
-         <slip1>0.5</slip1>
-         <slip2>0</slip2>
-         <material>Gazebo/Black</material>
+      <gazebo reference="${fb}_${lr}_wheel">
+         <material>Gazebo/Blue</material>
          <turnGravityOff>false</turnGravityOff>
       </gazebo>
@@ -47,5 +82,5 @@
          <parent link="${parent}"/>
          <child link="${fb}_${lr}_wheel" />
-         <origin xyz="${translateX} ${translateY} ${translateZ}" rpy="0 0 0" />
+         <origin xyz="${translateX} ${translateY} ${translateZ}" rpy="${flipY * 1 * DEG_TO_RAD} 0 0" />
          <limit effort="1000" velocity="1000" />
          <axis xyz="0 1 0" />
@@ -54,14 +89,14 @@
       </joint>
       <!-- Transmission is important to link the joint and the controller -->
-      <transmission name="${fb}_${lr}_wheel_joint_trans" >
+      <transmission name="${fb}_${lr}_wheel_joint_trans">
          <type>transmission_interface/SimpleTransmission</type>
          <joint name="${fb}_${lr}_wheel_joint">
-            <hardwareInterface>hardware_interface/EffortJointInterface</hardwareInterface>
+            <hardwareInterface>hardware_interface/VelocityJointInterface</hardwareInterface>
          </joint>
          <actuator name="${fb}_${lr}_wheel_joint_motor">
-            <hardwareInterface>hardware_interface/EffortJointInterface</hardwareInterface>
-            <mechanicalReduction>1</mechanicalReduction> <!-- It is not true: we uses motor with gearbox and ration of 75 -->
+            <mechanicalReduction>1</mechanicalReduction>            <!-- It is not true: we uses motor with gearbox and ration of 75 -->
          </actuator>
       </transmission>
+      <xacro:grouser links_qty="20" max_qty="20" parent="${fb}_${lr}_wheel" flipY="${flipY}" flipZ="${flipZ}"/>
    </xacro:macro>
 </robot>

Commit message: rename robot and change filename

File: rover_config/urdf/rover.xacro (robot description, xacro)
@@ -1,6 +1,6 @@
 <?xml version="1.0"?>
-<robot name="test"
+<robot name="nimrod"
    xmlns:xacro="http://www.ros.org/wiki/xacro">
-   <xacro:include filename="$(find rover_config)/urdf/wheel.urdf.xacro" />
+   <xacro:include filename="$(find rover_config)/urdf/wheel.xacro" />
    <!-- Defining the colors used in this robot -->
    <material name="Black">
@@ -43,5 +43,5 @@
    <!-- It is necessary as gazebo does not support inertia for the root link -->
    <!-- Do not call it world as it is reserved for robot that must be fixed to the world -->
-  <link name="base_link">
+   <link name="base_link">
    </link>
    <gazebo reference="base_link">
@@ -124,32 +124,4 @@
    <rocker side="left" parent="chassis" translateX="0" translateY="${base_width / 2}" translateZ="${-base_height / 3}" flipY="1" />
    <rocker side="right" parent="chassis" translateX="0" translateY="${-base_width / 2}" translateZ="${-base_height / 3}" flipY="-1" />
-   <!-- Wheel Definition for simulation -->
-   <!-- <wheel fb="front" lr="right" parent="chassis" translateX="0.4" translateY="${-1*(base_width/2+0.04)}" translateZ="-0.065" flipY="1"/>
-   <wheel fb="front" lr="left" parent="chassis" translateX="0.4" translateY="${1*(base_width/2+0.04)}" translateZ="-0.065" flipY="1"/>
-   <wheel fb="back" lr="right" parent="chassis" translateX="-0.4" translateY="${-1*(base_width/2+0.04)}" translateZ="-0.065" flipY="1"/>
-   <wheel fb="back" lr="left" parent="chassis" translateX="-0.4" translateY="${1*(base_width/2+0.04)}" translateZ="-0.065" flipY="1"/> -->
-   <!-- Skid Steering Drive for 4 wheel robot for simulation -->
-   <!-- <gazebo>
-      <plugin name="drive_controller" filename="libgazebo_ros_skid_steer_drive.so">
-         <updateRate>100</updateRate>
-         <robotNameSpace>/</robotNameSpace>
-         <leftFrontJoint>front_left_wheel_joint</leftFrontJoint>
-         <rightFrontJoint>front_right_wheel_joint</rightFrontJoint>
-         <leftRearJoint>back_left_wheel_joint</leftRearJoint>
-         <rightRearJoint>back_right_wheel_joint</rightRearJoint>
-         <wheelSeparation>${rocker_lenght}</wheelSeparation>
-         <wheelDiameter>0.32</wheelDiameter>
-         <robotBaseFrame>base_link</robotBaseFrame>
-         <torque>100</torque>
-         <topicName>cmd_vel</topicName>
-         <broadcastTF>true</broadcastTF>
-         <commandTopic>cmd_vel</commandTopic>
-         <odometryTopic>odom</odometryTopic>
-         <odometryFrame>odom</odometryFrame>
-         <covariance_x>0.00100</covariance_x>
-         <covariance_y>0.00100</covariance_y>
-         <covariance_yaw>0.010000</covariance_yaw>
-      </plugin>
-   </gazebo> -->
    <!-- Publishing joint states from Gazebo simulator -->
    <!-- fixed links are not published -->

Commit message: rudimentary gazebo camera and IMU sensors

File: rover_config/urdf/rover.xacro (robot description, xacro)
@@ -31,4 +31,5 @@
    <xacro:property name="rocker_mass" value="2.0" />
    <xacro:property name="rocker_offsetZ" value="0.2" />
+   <xacro:property name="camera_size" value="0.05" />
    <!-- Macro for calculating inertia of cylinder -->
    <xacro:macro name="cylinder_inertia" params="m r h">
@@ -124,4 +125,90 @@
    <rocker side="left" parent="chassis" translateX="0" translateY="${base_width / 2}" translateZ="${-base_height / 3}" flipY="1" />
    <rocker side="right" parent="chassis" translateX="0" translateY="${-base_width / 2}" translateZ="${-base_height / 3}" flipY="-1" />
+   <!-- Camera gazebo sensor -->
+   <joint name="camera_joint" type="fixed">
+    <axis xyz="0 1 0" />
+    <origin xyz="${base_lenght / 2 + 2 * camera_size} 0 ${base_height / 2}" rpy="0 0 0"/>
+    <parent link="chassis"/>
+    <child link="camera_link"/>
+  </joint>
+  <link name="camera_link">
+    <collision>
+      <origin xyz="0 0 0" rpy="0 0 0"/>
+      <geometry>
+    <box size="${camera_size} ${camera_size} ${camera_size}"/>
+      </geometry>
+    </collision>
+    <visual>
+      <origin xyz="0 0 0" rpy="0 0 0"/>
+      <geometry>
+    <box size="${camera_size} ${camera_size} ${camera_size}"/>
+      </geometry>
+      <material name="red"/>
+    </visual>
+    <inertial>
+      <mass value="1e-5" />
+      <origin xyz="0 0 0" rpy="0 0 0"/>
+      <inertia ixx="1e-6" ixy="0" ixz="0" iyy="1e-6" iyz="0" izz="1e-6" />
+    </inertial>
+  </link>
+  <gazebo reference="camera_link">
+    <sensor type="camera" name="camera1">
+      <update_rate>30.0</update_rate>
+      <camera name="head">
+        <horizontal_fov>1.3962634</horizontal_fov>
+        <image>
+          <width>800</width>
+          <height>800</height>
+          <format>R8G8B8</format>
+        </image>
+        <clip>
+          <near>0.02</near>
+          <far>300</far>
+        </clip>
+        <noise>
+          <type>gaussian</type>
+          <!-- Noise is sampled independently per pixel on each frame.
+               That pixel's noise value is added to each of its color
+               channels, which at that point lie in the range [0,1]. -->
+          <mean>0.0</mean>
+          <stddev>0.007</stddev>
+        </noise>
+      </camera>
+      <plugin name="camera_controller" filename="libgazebo_ros_camera.so">
+        <alwaysOn>true</alwaysOn>
+        <updateRate>0.0</updateRate>
+        <cameraName>rrbot/camera1</cameraName>
+        <imageTopicName>image_raw</imageTopicName>
+        <cameraInfoTopicName>camera_info</cameraInfoTopicName>
+        <frameName>camera_link</frameName>
+        <hackBaseline>0.07</hackBaseline>
+        <distortionK1>0.0</distortionK1>
+        <distortionK2>0.0</distortionK2>
+        <distortionK3>0.0</distortionK3>
+        <distortionT1>0.0</distortionT1>
+        <distortionT2>0.0</distortionT2>
+      </plugin>
+    </sensor>
+  </gazebo>
+  <!-- IMU gazebo sensor -->
+  <gazebo reference="chassis">
+    <gravity>true</gravity>
+    <sensor name="imu_sensor" type="imu">
+      <always_on>true</always_on>
+      <update_rate>100</update_rate>
+      <visualize>true</visualize>
+      <topic>__default_topic__</topic>
+      <plugin filename="libgazebo_ros_imu_sensor.so" name="imu_plugin">
+        <topicName>imu</topicName>
+        <bodyName>chassis</bodyName>
+        <updateRateHZ>10.0</updateRateHZ>
+        <gaussianNoise>0.0</gaussianNoise>
+        <xyzOffset>0 0 0</xyzOffset>
+        <rpyOffset>0 0 0</rpyOffset>
+        <frameName>chassis</frameName>
+      </plugin>
+      <pose>0 0 0 0 0 0</pose>
+    </sensor>
+  </gazebo>
    <!-- Publishing joint states from Gazebo simulator -->
    <!-- fixed links are not published -->
