Commit message: Add new camera_link to compensate rotation

File: rover_config/urdf/rover.xacro (robot description, xacro)
@@ -1,233 +1,241 @@
 <?xml version="1.0"?>
 <robot name="nimrod"
-   xmlns:xacro="http://www.ros.org/wiki/xacro">
-   <xacro:include filename="$(find rover_config)/urdf/wheel.xacro" />
-   <!-- Defining the colors used in this robot -->
-   <material name="Black">
-      <color rgba="0.0 0.0 0.0 1.0"/>
-   </material>
-   <material name="Red">
-      <color rgba="0.8 0.0 0.0 1.0"/>
-   </material>
-   <material name="White">
-      <color rgba="1.0 1.0 1.0 1.0"/>
-   </material>
-   <material name="Blue">
-      <color rgba="0.0 0.0 0.8 1.0"/>
-   </material>
-   <!-- Property list -->
-   <!-- All units in m-kg-s-radians unit system -->
-   <xacro:property name="M_PI" value="3.1415926535897931" />
-   <xacro:property name="M_PI_2" value="1.570796327" />
-   <xacro:property name="DEG_TO_RAD" value="0.017453293" />
-   <!-- Main body length height width -->
-   <xacro:property name="base_height" value="0.2" />
-   <xacro:property name="base_width" value="0.2" />
-   <xacro:property name="base_lenght" value="0.5" />
-   <xacro:property name="base_mass" value="20.0" />
-   <xacro:property name="rocker_height" value="0.1" />
-   <xacro:property name="rocker_width" value="0.1" />
-   <xacro:property name="rocker_lenght" value="0.7" />
-   <xacro:property name="rocker_mass" value="2.0" />
-   <xacro:property name="rocker_offsetZ" value="0.2" />
-   <xacro:property name="camera_size" value="0.05" />
-   <!-- Macro for calculating inertia of cylinder -->
-   <xacro:macro name="cylinder_inertia" params="m r h">
-      <inertia ixx="${ m * ( 3 * r*r + h*h ) / 12}" ixy="0" ixz="0" iyy="${ m * ( 3 * r*r + h*h ) / 12}" iyz="0" izz="${ m * r / 2}" />
-   </xacro:macro>
-   <!-- Macro for calculating inertia of a box -->
-   <xacro:macro name="box_inertia" params="m x y z">
-      <inertia ixx="${0.0833333 * m * (y*y + z*z)}" ixy="0.0" ixz="0.0" iyy="${0.0833333 * m * (x*x + z*z)}" iyz="0.0" izz="${0.0833333 * m * (x*x + y*y)}" />
-   </xacro:macro>
-   <!-- World link -->
-   <!-- base_footprint is a fictious link(frame) that is on the ground right below base_link origin -->
-   <!-- It is necessary as gazebo does not support inertia for the root link -->
-   <!-- Do not call it world as it is reserved for robot that must be fixed to the world -->
-   <link name="base_link">
-   </link>
-   <gazebo reference="base_link">
-      <turnGravityOff>false</turnGravityOff>
-   </gazebo>
-   <joint name="glue_robot_to_world" type="fixed">
-      <origin xyz="0 0 0.1" rpy="0 0 0" />
-      <parent link="base_link" />
-      <child link="chassis" />
-   </joint>
-   <!-- Base link -->
-   <!-- Actual body/chassis of the robot -->
-   <link name="chassis">
-      <inertial>
-         <mass value="${base_mass}" />
-         <!-- the3x3 rotational inertia matrix -->
-         <box_inertia m="${base_mass}" x="${base_lenght}" y="${base_width}" z="${base_height}" />
-         <origin xyz="0 0 0" />
-      </inertial>
-      <visual>
-         <origin xyz="0 0 0" rpy="0 0 0" />
-         <geometry>
-            <box size="${base_lenght} ${base_width} ${base_height}" />
-         </geometry>
-         <material name="Blue" />
-      </visual>
-      <collision>
-         <origin xyz="0 0 0" rpy="0 0 0" />
-         <geometry>
-            <box size="${base_lenght} ${base_width} ${base_height}" />
-         </geometry>
-      </collision>
-   </link>
-   <gazebo reference="chassis">
-      <material>Gazebo/White</material>
-      <turnGravityOff>false</turnGravityOff>
-   </gazebo>
-   <xacro:macro name="rocker" params="side parent translateX translateY translateZ flipY">
-      <link name="${side}_rocker">
-         <visual>
-            <origin xyz="0 ${flipY * rocker_width / 2} ${-rocker_offsetZ}" rpy="0 0 0"/>
-            <geometry>
-               <box size="${rocker_lenght} ${rocker_width} ${rocker_height}" />
-            </geometry>
-            <material name="Red" />
-         </visual>
-         <collision>
-            <origin xyz="0 ${flipY * rocker_width / 2} ${-rocker_offsetZ}" rpy="0 0 0"/>
-            <geometry>
-               <box size="${rocker_lenght} ${rocker_width} ${rocker_height}" />
-            </geometry>
-         </collision>
-         <inertial>
-            <mass value="${rocker_mass}" />
-            <origin xyz="0 ${flipY * rocker_width / 2} ${-rocker_offsetZ}" rpy="0 0 0"/>
-            <box_inertia m="${rocker_mass}" x="${rocker_lenght}" y="${rocker_width}" z="${rocker_height}" />
-         </inertial>
-      </link>
-      <joint name="${side}_rocker_joint" type="revolute">
-         <origin xyz="${translateX} ${translateY} ${translateZ}" rpy="0.0 0.0 0.0"/>
-         <parent link="${parent}"/>
-         <child link="${side}_rocker"/>
-         <axis xyz="0 1 0"/>
-         <dynamics damping="0" friction="0.5"/>
-         <limit lower="${-30 * DEG_TO_RAD}" upper="${30 * DEG_TO_RAD}" velocity="1000" effort="1000"/>
-      </joint>
-      <transmission name="${side}_rocker_joint_trans">
-         <type>transmission_interface/SimpleTransmission</type>
-         <joint name="${side}_rocker_joint">
-            <hardwareInterface>hardware_interface/PositionJointInterface</hardwareInterface>
-         </joint>
-         <actuator name="${side}_rocker_joint_motor">
-            <hardwareInterface>hardware_interface/PositionJointInterface</hardwareInterface>
-            <mechanicalReduction>1</mechanicalReduction>
-         </actuator>
-      </transmission>
-      <wheel fb="front" lr="${side}" parent="${side}_rocker" translateX="${rocker_lenght / 2}" translateY="${flipY * rocker_width}" translateZ="${-rocker_offsetZ -rocker_height / 2}" flipY="${flipY}" flipZ="1"/>
-      <wheel fb="back" lr="${side}" parent="${side}_rocker" translateX="${-rocker_lenght / 2}" translateY="${flipY * rocker_width}" translateZ="${-rocker_offsetZ -rocker_height / 2}" flipY="${flipY}" flipZ="-1"/>
-   </xacro:macro>
-   <rocker side="left" parent="chassis" translateX="0" translateY="${base_width / 2}" translateZ="${-base_height / 3}" flipY="1" />
-   <rocker side="right" parent="chassis" translateX="0" translateY="${-base_width / 2}" translateZ="${-base_height / 3}" flipY="-1" />
-   <!-- Camera gazebo sensor -->
-   <joint name="camera_joint" type="fixed">
-    <axis xyz="0 1 0" />
-    <origin xyz="${base_lenght / 2 + 2 * camera_size} 0 ${base_height / 2}" rpy="0 0 0"/>
-    <parent link="chassis"/>
-    <child link="camera_link"/>
-  </joint>
-  <link name="camera_link">
-    <collision>
-      <origin xyz="0 0 0" rpy="0 0 0"/>
-      <geometry>
-    <box size="${camera_size} ${camera_size} ${camera_size}"/>
-      </geometry>
-    </collision>
-    <visual>
-      <origin xyz="0 0 0" rpy="0 0 0"/>
-      <geometry>
-    <box size="${camera_size} ${camera_size} ${camera_size}"/>
-      </geometry>
-      <material name="red"/>
-    </visual>
-    <inertial>
-      <mass value="1e-5" />
-      <origin xyz="0 0 0" rpy="0 0 0"/>
-      <inertia ixx="1e-6" ixy="0" ixz="0" iyy="1e-6" iyz="0" izz="1e-6" />
-    </inertial>
-  </link>
-  <gazebo reference="camera_link">
-    <sensor type="camera" name="camera1">
-      <update_rate>30.0</update_rate>
-      <camera name="head">
-        <horizontal_fov>1.3962634</horizontal_fov>
-        <image>
-          <width>800</width>
-          <height>800</height>
-          <format>R8G8B8</format>
-        </image>
-        <clip>
-          <near>0.02</near>
-          <far>300</far>
-        </clip>
-        <noise>
-          <type>gaussian</type>
-          <!-- Noise is sampled independently per pixel on each frame.
+    xmlns:xacro="http://www.ros.org/wiki/xacro">
+    <xacro:include filename="$(find rover_config)/urdf/wheel.xacro" />
+    <!-- Defining the colors used in this robot -->
+    <material name="Black">
+        <color rgba="0.0 0.0 0.0 1.0"/>
+    </material>
+    <material name="Red">
+        <color rgba="0.8 0.0 0.0 1.0"/>
+    </material>
+    <material name="White">
+        <color rgba="1.0 1.0 1.0 1.0"/>
+    </material>
+    <material name="Blue">
+        <color rgba="0.0 0.0 0.8 1.0"/>
+    </material>
+    <!-- Property list -->
+    <!-- All units in m-kg-s-radians unit system -->
+    <xacro:property name="M_PI" value="3.1415926535897931" />
+    <xacro:property name="M_PI_2" value="1.570796327" />
+    <xacro:property name="DEG_TO_RAD" value="0.017453293" />
+    <!-- Main body length height width -->
+    <xacro:property name="base_height" value="0.2" />
+    <xacro:property name="base_width" value="0.2" />
+    <xacro:property name="base_lenght" value="0.5" />
+    <xacro:property name="base_mass" value="20.0" />
+    <xacro:property name="rocker_height" value="0.1" />
+    <xacro:property name="rocker_width" value="0.1" />
+    <xacro:property name="rocker_lenght" value="0.7" />
+    <xacro:property name="rocker_mass" value="2.0" />
+    <xacro:property name="rocker_offsetZ" value="0.2" />
+    <xacro:property name="camera_size" value="0.05" />
+    <!-- Macro for calculating inertia of cylinder -->
+    <xacro:macro name="cylinder_inertia" params="m r h">
+        <inertia ixx="${ m * ( 3 * r*r + h*h ) / 12}" ixy="0" ixz="0" iyy="${ m * ( 3 * r*r + h*h ) / 12}" iyz="0" izz="${ m * r / 2}" />
+    </xacro:macro>
+    <!-- Macro for calculating inertia of a box -->
+    <xacro:macro name="box_inertia" params="m x y z">
+        <inertia ixx="${0.0833333 * m * (y*y + z*z)}" ixy="0.0" ixz="0.0" iyy="${0.0833333 * m * (x*x + z*z)}" iyz="0.0" izz="${0.0833333 * m * (x*x + y*y)}" />
+    </xacro:macro>
+    <!-- World link -->
+    <!-- base_footprint is a fictious link(frame) that is on the ground right below base_link origin -->
+    <!-- It is necessary as gazebo does not support inertia for the root link -->
+    <!-- Do not call it world as it is reserved for robot that must be fixed to the world -->
+    <link name="base_link">
+    </link>
+    <gazebo reference="base_link">
+        <turnGravityOff>false</turnGravityOff>
+    </gazebo>
+    <joint name="glue_robot_to_world" type="fixed">
+        <origin xyz="0 0 0.1" rpy="0 0 0" />
+        <parent link="base_link" />
+        <child link="chassis" />
+    </joint>
+    <!-- Base link -->
+    <!-- Actual body/chassis of the robot -->
+    <link name="chassis">
+        <inertial>
+            <mass value="${base_mass}" />
+            <!-- the3x3 rotational inertia matrix -->
+            <box_inertia m="${base_mass}" x="${base_lenght}" y="${base_width}" z="${base_height}" />
+            <origin xyz="0 0 0" />
+        </inertial>
+        <visual>
+            <origin xyz="0 0 0" rpy="0 0 0" />
+            <geometry>
+                <box size="${base_lenght} ${base_width} ${base_height}" />
+            </geometry>
+            <material name="Blue" />
+        </visual>
+        <collision>
+            <origin xyz="0 0 0" rpy="0 0 0" />
+            <geometry>
+                <box size="${base_lenght} ${base_width} ${base_height}" />
+            </geometry>
+        </collision>
+    </link>
+    <gazebo reference="chassis">
+        <material>Gazebo/White</material>
+        <turnGravityOff>false</turnGravityOff>
+    </gazebo>
+    <xacro:macro name="rocker" params="side parent translateX translateY translateZ flipY">
+        <link name="${side}_rocker">
+            <visual>
+                <origin xyz="0 ${flipY * rocker_width / 2} ${-rocker_offsetZ}" rpy="0 0 0"/>
+                <geometry>
+                    <box size="${rocker_lenght} ${rocker_width} ${rocker_height}" />
+                </geometry>
+                <material name="Red" />
+            </visual>
+            <collision>
+                <origin xyz="0 ${flipY * rocker_width / 2} ${-rocker_offsetZ}" rpy="0 0 0"/>
+                <geometry>
+                    <box size="${rocker_lenght} ${rocker_width} ${rocker_height}" />
+                </geometry>
+            </collision>
+            <inertial>
+                <mass value="${rocker_mass}" />
+                <origin xyz="0 ${flipY * rocker_width / 2} ${-rocker_offsetZ}" rpy="0 0 0"/>
+                <box_inertia m="${rocker_mass}" x="${rocker_lenght}" y="${rocker_width}" z="${rocker_height}" />
+            </inertial>
+        </link>
+        <joint name="${side}_rocker_joint" type="revolute">
+            <origin xyz="${translateX} ${translateY} ${translateZ}" rpy="0.0 0.0 0.0"/>
+            <parent link="${parent}"/>
+            <child link="${side}_rocker"/>
+            <axis xyz="0 1 0"/>
+            <dynamics damping="0" friction="0.5"/>
+            <limit lower="${-30 * DEG_TO_RAD}" upper="${30 * DEG_TO_RAD}" velocity="1000" effort="1000"/>
+        </joint>
+        <transmission name="${side}_rocker_joint_trans">
+            <type>transmission_interface/SimpleTransmission</type>
+            <joint name="${side}_rocker_joint">
+                <hardwareInterface>hardware_interface/PositionJointInterface</hardwareInterface>
+            </joint>
+            <actuator name="${side}_rocker_joint_motor">
+                <hardwareInterface>hardware_interface/PositionJointInterface</hardwareInterface>
+                <mechanicalReduction>1</mechanicalReduction>
+            </actuator>
+        </transmission>
+        <wheel fb="front" lr="${side}" parent="${side}_rocker" translateX="${rocker_lenght / 2}" translateY="${flipY * rocker_width}" translateZ="${-rocker_offsetZ -rocker_height / 2}" flipY="${flipY}" flipZ="1"/>
+        <wheel fb="back" lr="${side}" parent="${side}_rocker" translateX="${-rocker_lenght / 2}" translateY="${flipY * rocker_width}" translateZ="${-rocker_offsetZ -rocker_height / 2}" flipY="${flipY}" flipZ="-1"/>
+    </xacro:macro>
+    <rocker side="left" parent="chassis" translateX="0" translateY="${base_width / 2}" translateZ="${-base_height / 3}" flipY="1" />
+    <rocker side="right" parent="chassis" translateX="0" translateY="${-base_width / 2}" translateZ="${-base_height / 3}" flipY="-1" />
+    <!-- Camera gazebo sensor -->
+    <joint name="camera_joint" type="fixed">
+        <axis xyz="0 1 0" />
+        <origin xyz="${base_lenght / 2 + 2 * camera_size} 0 ${base_height / 2}" rpy="0 0 0"/>
+        <parent link="chassis"/>
+        <child link="camera_link"/>
+    </joint>
+    <link name="camera_link">
+        <collision>
+            <origin xyz="0 0 0" rpy="0 0 0"/>
+            <geometry>
+                <box size="${camera_size} ${camera_size} ${camera_size}"/>
+            </geometry>
+        </collision>
+        <visual>
+            <origin xyz="0 0 0" rpy="0 0 0"/>
+            <geometry>
+                <box size="${camera_size} ${camera_size} ${camera_size}"/>
+            </geometry>
+            <material name="red"/>
+        </visual>
+        <inertial>
+            <mass value="1e-5" />
+            <origin xyz="0 0 0" rpy="0 0 0"/>
+            <inertia ixx="1e-6" ixy="0" ixz="0" iyy="1e-6" iyz="0" izz="1e-6" />
+        </inertial>
+    </link>
+    <link name="camera_link2">
+    </link>
+    <joint name="camera_joint2" type="fixed">
+        <axis xyz="0 1 0" />
+        <origin xyz="0 0 0" rpy="${-M_PI_2} 0 ${-M_PI_2}"/>
+        <parent link="camera_link"/>
+        <child link="camera_link2"/>
+    </joint>
+    <gazebo reference="camera_link">
+        <sensor type="camera" name="camera1">
+            <update_rate>30.0</update_rate>
+            <camera name="head">
+                <horizontal_fov>1.3962634</horizontal_fov>
+                <image>
+                    <width>800</width>
+                    <height>800</height>
+                    <format>R8G8B8</format>
+                </image>
+                <clip>
+                    <near>0.02</near>
+                    <far>300</far>
+                </clip>
+                <noise>
+                    <type>gaussian</type>
+                    <!-- Noise is sampled independently per pixel on each frame.
                That pixel's noise value is added to each of its color
                channels, which at that point lie in the range [0,1]. -->
-          <mean>0.0</mean>
-          <stddev>0.007</stddev>
-        </noise>
-      </camera>
-      <plugin name="camera_controller" filename="libgazebo_ros_camera.so">
-        <alwaysOn>true</alwaysOn>
-        <updateRate>0.0</updateRate>
-        <cameraName>sensors/camera1</cameraName>
-        <imageTopicName>image_raw</imageTopicName>
-        <cameraInfoTopicName>camera_info</cameraInfoTopicName>
-        <frameName>camera_link</frameName>
-        <hackBaseline>0.07</hackBaseline>
-        <distortionK1>0.0</distortionK1>
-        <distortionK2>0.0</distortionK2>
-        <distortionK3>0.0</distortionK3>
-        <distortionT1>0.0</distortionT1>
-        <distortionT2>0.0</distortionT2>
-      </plugin>
-    </sensor>
-  </gazebo>
-  <!-- IMU plugin sensor -->
-  <!-- computed by seperate plugin, without gravity -->
-  <gazebo>
-    <plugin name="imu_plugin" filename="libgazebo_ros_imu.so">
-      <alwaysOn>true</alwaysOn>
-      <bodyName>chassis</bodyName>
-      <topicName>sensors/imu_plugin</topicName>
-      <serviceName>imu_service</serviceName>
-      <gaussianNoise>0.0</gaussianNoise>
-      <updateRate>20.0</updateRate>
-    </plugin>
-  </gazebo>
-  <!-- IMU gazebo sensor -->
-  <!-- computed by gazebo, with gravity -->
-  <gazebo reference="chassis">
-    <gravity>true</gravity>
-    <sensor name="imu_sensor" type="imu">
-      <always_on>true</always_on>
-      <update_rate>50</update_rate>
-      <visualize>true</visualize>
-      <topic>__default_topic__</topic>
-      <plugin filename="libgazebo_ros_imu_sensor.so" name="imu_plugin">
-        <topicName>sensors/imu_gazebo</topicName>
-        <bodyName>chassis</bodyName>
-        <updateRateHZ>20.0</updateRateHZ>
-        <gaussianNoise>0.0</gaussianNoise>
-        <xyzOffset>0 0 0</xyzOffset>
-        <rpyOffset>0 0 0</rpyOffset>
-        <frameName>chassis</frameName>
-      </plugin>
-      <pose>0 0 0 0 0 0</pose>
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