Commit message: Add CAD Model of Rover

File: rover_config/urdf/rover.xacro (robot description, xacro)
@@ -30,5 +30,5 @@
     <xacro:property name="rocker_lenght" value="0.7" />
     <xacro:property name="rocker_mass" value="2.0" />
-    <xacro:property name="rocker_offsetZ" value="0.2" />
+    <xacro:property name="rocker_offsetZ" value="0" />
     <xacro:property name="camera_size" value="0.05" />
     <!-- Macro for calculating inertia of cylinder -->
@@ -64,19 +64,20 @@
         </inertial>
         <visual>
-            <origin xyz="0 0 0" rpy="0 0 0" />
+            <origin xyz="0 0 0" rpy="0 0 ${-90 * DEG_TO_RAD}" />
             <geometry>
-                <box size="${base_lenght} ${base_width} ${base_height}" />
+                <mesh filename="package://rover_config/rover_collada/Body_lowPoly.dae"/>
             </geometry>
-            <material name="Blue" />
+            <material name="Black" />
         </visual>
         <collision>
-            <origin xyz="0 0 0" rpy="0 0 0" />
+            <origin xyz="0 0 0" rpy="0 0 ${-90 * DEG_TO_RAD}" />
             <geometry>
-                <box size="${base_lenght} ${base_width} ${base_height}" />
+                <mesh filename="package://rover_config/rover_collada/Body_lowPoly.dae"/>
             </geometry>
+            <material name="Black" />
         </collision>
     </link>
     <gazebo reference="chassis">
-        <material>Gazebo/White</material>
+        <material>Gazebo/Black</material>
         <turnGravityOff>false</turnGravityOff>
     </gazebo>
@@ -84,15 +85,16 @@
         <link name="${side}_rocker">
             <visual>
-                <origin xyz="0 ${flipY * rocker_width / 2} ${-rocker_offsetZ}" rpy="0 0 0"/>
+                <origin xyz="0 0 ${-rocker_offsetZ}" rpy="0 0 ${-90 * DEG_TO_RAD}"/>
                 <geometry>
-                    <box size="${rocker_lenght} ${rocker_width} ${rocker_height}" />
+                    <mesh filename="package://rover_config/rover_collada/Rocker_lowPoly.dae" scale="${flipY} 1 1"/>
                 </geometry>
-                <material name="Red" />
+                <material name="Blue" />
             </visual>
             <collision>
-                <origin xyz="0 ${flipY * rocker_width / 2} ${-rocker_offsetZ}" rpy="0 0 0"/>
+                <origin xyz="0 0 ${-rocker_offsetZ}" rpy="0 0 ${-90 * DEG_TO_RAD}"/>
                 <geometry>
-                    <box size="${rocker_lenght} ${rocker_width} ${rocker_height}" />
+                    <mesh filename="package://rover_config/rover_collada/Rocker_lowPoly.dae" scale="${flipY} 1 1"/>
                 </geometry>
+                <material name="Blue" />
             </collision>
             <inertial>
@@ -108,5 +110,5 @@
             <axis xyz="0 1 0"/>
             <dynamics damping="0" friction="0.5"/>
-            <limit lower="${-30 * DEG_TO_RAD}" upper="${30 * DEG_TO_RAD}" velocity="1000" effort="1000"/>
+            <limit lower="${-8 * DEG_TO_RAD}" upper="${8 * DEG_TO_RAD}" velocity="1000" effort="1000"/>
         </joint>
         <transmission name="${side}_rocker_joint_trans">
@@ -120,9 +122,13 @@
             </actuator>
         </transmission>
-        <wheel fb="front" lr="${side}" parent="${side}_rocker" translateX="${rocker_lenght / 2}" translateY="${flipY * rocker_width}" translateZ="${-rocker_offsetZ -rocker_height / 2}" flipY="${flipY}" flipZ="1"/>
-        <wheel fb="back" lr="${side}" parent="${side}_rocker" translateX="${-rocker_lenght / 2}" translateY="${flipY * rocker_width}" translateZ="${-rocker_offsetZ -rocker_height / 2}" flipY="${flipY}" flipZ="-1"/>
+        <wheel fb="front" lr="${side}" parent="${side}_rocker" translateX="0.350" translateY="${flipY * 0.300}" translateZ="-0.100" flipY="${flipY}" flipZ="1"/>
+        <wheel fb="back" lr="${side}" parent="${side}_rocker" translateX="-0.350" translateY="${flipY * 0.300}" translateZ="-0.100" flipY="${flipY}" flipZ="-1"/>
+        <gazebo reference="${side}_rocker">
+            <material>Gazebo/Blue</material>
+            <turnGravityOff>false</turnGravityOff>
+        </gazebo>
     </xacro:macro>
-    <rocker side="left" parent="chassis" translateX="0" translateY="${base_width / 2}" translateZ="${-base_height / 3}" flipY="1" />
-    <rocker side="right" parent="chassis" translateX="0" translateY="${-base_width / 2}" translateZ="${-base_height / 3}" flipY="-1" />
+    <rocker side="left" parent="chassis" translateX="0" translateY="0" translateZ="0" flipY="1" />
+    <rocker side="right" parent="chassis" translateX="0" translateY="0" translateZ="0" flipY="-1" />
     <!-- Camera gazebo sensor -->
     <joint name="camera_joint" type="fixed">
@@ -133,22 +139,4 @@
     </joint>
     <link name="camera_link">
-        <collision>
-            <origin xyz="0 0 0" rpy="0 0 0"/>
-            <geometry>
-                <box size="${camera_size} ${camera_size} ${camera_size}"/>
-            </geometry>
-        </collision>
-        <visual>
-            <origin xyz="0 0 0" rpy="0 0 0"/>
-            <geometry>
-                <box size="${camera_size} ${camera_size} ${camera_size}"/>
-            </geometry>
-            <material name="red"/>
-        </visual>
-        <inertial>
-            <mass value="1e-5" />
-            <origin xyz="0 0 0" rpy="0 0 0"/>
-            <inertia ixx="1e-6" ixy="0" ixz="0" iyy="1e-6" iyz="0" izz="1e-6" />
-        </inertial>
     </link>
     <link name="camera_link2">

File: rover_config/urdf/wheel.xacro (robot description, xacro)
@@ -2,5 +2,5 @@
 <robot name="wheel"
     xmlns:xacro="http://www.ros.org/wiki/xacro">
-    <xacro:property name="wheel_radius" value="0.15" />
+    <xacro:property name="wheel_radius" value="0.14" />
     <xacro:property name="wheel_width" value="0.2" />
     <xacro:property name="wheel_mass" value="1" />
@@ -13,17 +13,17 @@
     <xacro:macro name="grouser" params="links_qty max_qty parent flipY flipZ">
         <link name="${flipY}${flipZ}_${links_qty}">
-            <visual>
-                <origin xyz="0 ${flipY * wheel_width / 2} ${wheel_radius}" rpy="0 0 ${flipY * flipZ * 30 * DEG_TO_RAD}"/>
+            <!-- <visual>
+                <origin xyz="0 0 ${wheel_radius - 0.025}" rpy="0 0 ${flipY * flipZ * 30 * DEG_TO_RAD}"/>
                 <geometry>
                     <box size="0.01 ${wheel_width} 0.05"/>
                 </geometry>
-                <material name="Red" />
-            </visual>
+                <material name="Black" />
+            </visual> -->
             <collision>
-                <origin xyz="0 ${flipY * wheel_width / 2} ${wheel_radius}" rpy="0 0 ${flipY * flipZ * 30 * DEG_TO_RAD}"/>
+                <origin xyz="0 0 ${wheel_radius - 0.025}" rpy="0 0 ${flipY * flipZ * 30 * DEG_TO_RAD}"/>
                 <geometry>
                     <box size="0.01 ${wheel_width} 0.05"/>
                 </geometry>
-                <material name="Red" />
+                <material name="Black" />
             </collision>
             <inertial>
@@ -39,9 +39,9 @@
         </joint>
         <gazebo reference="${flipY}${flipZ}_${links_qty}">
-            <mu1 value="10"/>
-            <mu2 value="0.1" />
+            <mu1 value="100000"/>
+            <mu2 value="0.25" />
             <!-- <mu2 value="1" /> -->
-            <!-- <fdir1 value="0.7071 ${-flipY * flipZ * 0.7071} 0" /> -->
-            <fdir1 value="1 0 0" />
+            <fdir1 value="0.7071 ${-flipY * flipZ * 0.7071} 0" />
+            <!-- <fdir1 value="1 0 0" /> -->
             <kp value="10000000.0" />
             <kd value="1.0" />
@@ -57,15 +57,15 @@
         <link name="${fb}_${lr}_wheel">
             <visual>
-                <origin xyz="0 ${flipY * wheel_width / 2} 0" rpy="${flipY*M_PI/2} 0 0"/>
+                <origin xyz="0 0 0" rpy="0 0 ${-90 * DEG_TO_RAD}"/>
                 <!-- make sure the wheel is in the correct position -->
                 <geometry>
-                    <cylinder length="${wheel_width}" radius="${wheel_radius}" />
+                    <mesh filename="package://rover_config/rover_collada/Wheel_lowPoly.dae" scale="${-flipY * flipZ} 1 1"/>
                 </geometry>
-                <material name="Black" />
+                <material name="Red" />
             </visual>
             <collision>
-                <origin xyz="0 ${flipY * wheel_width / 2} 0" rpy="${flipY*M_PI/2} 0 0"/>
+                <origin xyz="0 0 0" rpy="${flipY*M_PI/2} 0 0"/>
                 <geometry>
-                    <cylinder length="${wheel_width}" radius="${wheel_radius}" />
+                    <cylinder length="${wheel_width}" radius="${wheel_radius - 0.025}" />
                 </geometry>
             </collision>
@@ -77,5 +77,5 @@
         </link>
         <gazebo reference="${fb}_${lr}_wheel">
-            <material>Gazebo/Blue</material>
+            <material>Gazebo/Red</material>
             <turnGravityOff>false</turnGravityOff>
         </gazebo>

Commit message: Second camera configs

File: rover_config/urdf/rover.xacro (robot description, xacro)
@@ -187,4 +187,59 @@
         </sensor>
     </gazebo>
+    <joint name="camera2_joint" type="fixed">
+        <axis xyz="0 1 0" />
+        <origin xyz="${base_lenght / 2 + 2 * camera_size} 0 ${base_height / 2}" rpy="0 0 0"/>
+        <parent link="chassis"/>
+        <child link="camera2_link"/>
+    </joint>
+    <link name="camera2_link">
+    </link>
+    <link name="camera2_link2">
+    </link>
+    <joint name="camera2_joint2" type="fixed">
+        <axis xyz="0 1 0" />
+        <origin xyz="0 0 0" rpy="${-M_PI_2} 0 ${-M_PI_2}"/>
+        <parent link="camera2_link"/>
+        <child link="camera2_link2"/>
+    </joint>
+    <gazebo reference="camera2_link">
+        <sensor type="camera" name="camera2">
+            <update_rate>30.0</update_rate>
+            <camera name="head">
+                <horizontal_fov>${45 * DEG_TO_RAD}</horizontal_fov>
+                <image>
+                    <width>2056</width>
+                    <height>1542</height>
+                    <format>R8G8B8</format>
+                </image>
+                <clip>
+                    <near>0.02</near>
+                    <far>300</far>
+                </clip>
+                <noise>
+                    <type>gaussian</type>
+                    <!-- Noise is sampled independently per pixel on each frame.
+               That pixel's noise value is added to each of its color
+               channels, which at that point lie in the range [0,1]. -->
+                    <mean>0.0</mean>
+                    <stddev>0.07</stddev>
+                </noise>
+            </camera>
+            <plugin name="camera_controller" filename="libgazebo_ros_camera.so">
+                <alwaysOn>true</alwaysOn>
+                <updateRate>0.0</updateRate>
+                <cameraName>sensors/camera2</cameraName>
+                <imageTopicName>image_raw</imageTopicName>
+                <cameraInfoTopicName>camera2_info</cameraInfoTopicName>
+                <frameName>camera2_link2</frameName>
+                <hackBaseline>0.0</hackBaseline>
+                <distortionK1>0.0</distortionK1>
+                <distortionK2>0.0</distortionK2>
+                <distortionK3>0.0</distortionK3>
+                <distortionT1>0.0</distortionT1>
+                <distortionT2>0.0</distortionT2>
+            </plugin>
+        </sensor>
+    </gazebo>
     <!-- IMU plugin sensor -->
     <!-- computed by seperate plugin, without gravity -->

Commit message: Replaced one camera with two cameras with a wider FOV

File: rover_config/urdf/rover.xacro (robot description, xacro)
@@ -134,5 +134,5 @@
     <joint name="camera_joint" type="fixed">
         <axis xyz="0 1 0" />
-        <origin xyz="${base_lenght / 2 + 2 * camera_size} 0 ${base_height / 2}" rpy="0 0 0"/>
+        <origin xyz="${base_lenght / 2 + 2 * camera_size} -${base_lenght/5} ${base_height / 2}" rpy="0 0 0"/>
         <parent link="chassis"/>
         <child link="camera_link"/>
@@ -152,5 +152,5 @@
             <update_rate>30.0</update_rate>
             <camera name="head">
-                <horizontal_fov>${45 * DEG_TO_RAD}</horizontal_fov>
+                <horizontal_fov>${90 * DEG_TO_RAD}</horizontal_fov>
                 <image>
                     <width>2056</width>
@@ -189,5 +189,5 @@
     <joint name="camera2_joint" type="fixed">
         <axis xyz="0 1 0" />
-        <origin xyz="${base_lenght / 2 + 2 * camera_size} 0 ${base_height / 2}" rpy="0 0 0"/>
+        <origin xyz="${base_lenght / 2 + 2 * camera_size} ${base_lenght/5} ${base_height / 2}" rpy="0 0 0"/>
         <parent link="chassis"/>
         <child link="camera2_link"/>
@@ -207,5 +207,5 @@
             <update_rate>30.0</update_rate>
             <camera name="head">
-                <horizontal_fov>${45 * DEG_TO_RAD}</horizontal_fov>
+                <horizontal_fov>${90 * DEG_TO_RAD}</horizontal_fov>
                 <image>
                     <width>2056</width>

Commit message: Add Carbon Textures

File: rover_config/urdf/rover.xacro (robot description, xacro)
@@ -64,5 +64,5 @@
         </inertial>
         <visual>
-            <origin xyz="0 0 0" rpy="0 0 ${-90 * DEG_TO_RAD}" />
+            <origin xyz="0 0 0" rpy="0 0 ${radians(-90)}" />
             <geometry>
                 <mesh filename="package://rover_config/rover_collada/Body_lowPoly.dae"/>
@@ -71,5 +71,5 @@
         </visual>
         <collision>
-            <origin xyz="0 0 0" rpy="0 0 ${-90 * DEG_TO_RAD}" />
+            <origin xyz="0 0 0" rpy="0 0 ${radians(-90)}" />
             <geometry>
                 <mesh filename="package://rover_config/rover_collada/Body_lowPoly.dae"/>
@@ -79,5 +79,5 @@
     </link>
     <gazebo reference="chassis">
-        <material>Gazebo/Black</material>
+        <!-- <material>Gazebo/Black</material> -->
         <turnGravityOff>false</turnGravityOff>
     </gazebo>
@@ -125,5 +125,5 @@
         <wheel fb="back" lr="${side}" parent="${side}_rocker" translateX="-0.350" translateY="${flipY * 0.300}" translateZ="-0.100" flipY="${flipY}" flipZ="-1"/>
         <gazebo reference="${side}_rocker">
-            <material>Gazebo/Blue</material>
+            <!-- <material>Gazebo/Blue</material> -->
             <turnGravityOff>false</turnGravityOff>
         </gazebo>

File: rover_config/urdf/wheel.xacro (robot description, xacro)
@@ -77,5 +77,5 @@
         </link>
         <gazebo reference="${fb}_${lr}_wheel">
-            <material>Gazebo/Red</material>
+            <!-- <material>Gazebo/Red</material> -->
             <turnGravityOff>false</turnGravityOff>
         </gazebo>
