Commit message: split rover into body and config, removed old testarm (now in rover_arm)

File: rover_config/urdf/rover.xacro (robot description, xacro)
@@ -2,42 +2,5 @@
 <robot name="nimrod"
     xmlns:xacro="http://www.ros.org/wiki/xacro">
-    <xacro:include filename="$(find rover_config)/urdf/wheel.xacro" />
-    <!-- Defining the colors used in this robot -->
-    <material name="Black">
-        <color rgba="0.0 0.0 0.0 1.0"/>
-    </material>
-    <material name="Red">
-        <color rgba="0.8 0.0 0.0 1.0"/>
-    </material>
-    <material name="White">
-        <color rgba="1.0 1.0 1.0 1.0"/>
-    </material>
-    <material name="Blue">
-        <color rgba="0.0 0.0 0.8 1.0"/>
-    </material>
-    <!-- Property list -->
-    <!-- All units in m-kg-s-radians unit system -->
-    <xacro:property name="M_PI" value="3.1415926535897931" />
-    <xacro:property name="M_PI_2" value="1.570796327" />
-    <xacro:property name="DEG_TO_RAD" value="0.017453293" />
-    <!-- Main body length height width -->
-    <xacro:property name="base_height" value="0.2" />
-    <xacro:property name="base_width" value="0.2" />
-    <xacro:property name="base_lenght" value="0.5" />
-    <xacro:property name="base_mass" value="20.0" />
-    <xacro:property name="rocker_height" value="0.1" />
-    <xacro:property name="rocker_width" value="0.1" />
-    <xacro:property name="rocker_lenght" value="0.7" />
-    <xacro:property name="rocker_mass" value="2.0" />
-    <xacro:property name="rocker_offsetZ" value="0" />
-    <xacro:property name="camera_size" value="0.05" />
-    <!-- Macro for calculating inertia of cylinder -->
-    <xacro:macro name="cylinder_inertia" params="m r h">
-        <inertia ixx="${ m * ( 3 * r*r + h*h ) / 12}" ixy="0" ixz="0" iyy="${ m * ( 3 * r*r + h*h ) / 12}" iyz="0" izz="${ m * r / 2}" />
-    </xacro:macro>
-    <!-- Macro for calculating inertia of a box -->
-    <xacro:macro name="box_inertia" params="m x y z">
-        <inertia ixx="${0.0833333 * m * (y*y + z*z)}" ixy="0.0" ixz="0.0" iyy="${0.0833333 * m * (x*x + z*z)}" iyz="0.0" izz="${0.0833333 * m * (x*x + y*y)}" />
-    </xacro:macro>
+    <xacro:include filename="$(find rover_config)/urdf/body.xacro" />
     <!-- World link -->
     <!-- base_footprint is a fictious link(frame) that is on the ground right below base_link origin -->
@@ -49,175 +12,6 @@
         <turnGravityOff>false</turnGravityOff>
     </gazebo>
-    <joint name="glue_robot_to_world" type="fixed">
-        <origin xyz="0 0 0.1" rpy="0 0 0" />
-        <parent link="base_link" />
-        <child link="chassis" />
-    </joint>
-    <!-- Base link -->
-    <!-- Actual body/chassis of the robot -->
-    <link name="chassis">
-        <inertial>
-            <mass value="${base_mass}" />
-            <!-- the3x3 rotational inertia matrix -->
-            <box_inertia m="${base_mass}" x="${base_lenght}" y="${base_width}" z="${base_height}" />
-            <origin xyz="0 0 0" />
-        </inertial>
-        <visual>
-            <origin xyz="0 0 0" rpy="0 0 ${radians(-90)}" />
-            <geometry>
-                <mesh filename="package://rover_config/rover_collada/Body_lowPoly.dae"/>
-            </geometry>
-            <material name="Black" />
-        </visual>
-        <collision>
-            <origin xyz="0 0 0" rpy="0 0 ${radians(-90)}" />
-            <geometry>
-                <mesh filename="package://rover_config/rover_collada/Body_lowPoly.dae"/>
-            </geometry>
-            <material name="Black" />
-        </collision>
-    </link>
-    <gazebo reference="chassis">
-        <!-- <material>Gazebo/Black</material> -->
-        <turnGravityOff>false</turnGravityOff>
-    </gazebo>
-    <xacro:macro name="rocker" params="side parent translateX translateY translateZ flipY">
-        <link name="${side}_rocker">
-            <visual>
-                <origin xyz="0 0 ${-rocker_offsetZ}" rpy="0 0 ${-90 * DEG_TO_RAD}"/>
-                <geometry>
-                    <mesh filename="package://rover_config/rover_collada/Rocker_lowPoly.dae" scale="${flipY} 1 1"/>
-                </geometry>
-                <material name="Blue" />
-            </visual>
-            <collision>
-                <origin xyz="0 0 ${-rocker_offsetZ}" rpy="0 0 ${-90 * DEG_TO_RAD}"/>
-                <geometry>
-                    <mesh filename="package://rover_config/rover_collada/Rocker_lowPoly.dae" scale="${flipY} 1 1"/>
-                </geometry>
-                <material name="Blue" />
-            </collision>
-            <inertial>
-                <mass value="${rocker_mass}" />
-                <origin xyz="0 ${flipY * rocker_width / 2} ${-rocker_offsetZ}" rpy="0 0 0"/>
-                <box_inertia m="${rocker_mass}" x="${rocker_lenght}" y="${rocker_width}" z="${rocker_height}" />
-            </inertial>
-        </link>
-        <joint name="${side}_rocker_joint" type="revolute">
-            <origin xyz="${translateX} ${translateY} ${translateZ}" rpy="0.0 0.0 0.0"/>
-            <parent link="${parent}"/>
-            <child link="${side}_rocker"/>
-            <axis xyz="0 1 0"/>
-            <dynamics damping="0" friction="0.5"/>
-            <limit lower="${-8 * DEG_TO_RAD}" upper="${8 * DEG_TO_RAD}" velocity="1000" effort="1000"/>
-        </joint>
-        <transmission name="${side}_rocker_joint_trans">
-            <type>transmission_interface/SimpleTransmission</type>
-            <joint name="${side}_rocker_joint">
-                <hardwareInterface>hardware_interface/PositionJointInterface</hardwareInterface>
-            </joint>
-            <actuator name="${side}_rocker_joint_motor">
-                <hardwareInterface>hardware_interface/PositionJointInterface</hardwareInterface>
-                <mechanicalReduction>1</mechanicalReduction>
-            </actuator>
-        </transmission>
-        <wheel fb="front" lr="${side}" parent="${side}_rocker" translateX="0.350" translateY="${flipY * 0.300}" translateZ="-0.100" flipY="${flipY}" flipZ="1"/>
-        <wheel fb="back" lr="${side}" parent="${side}_rocker" translateX="-0.350" translateY="${flipY * 0.300}" translateZ="-0.100" flipY="${flipY}" flipZ="-1"/>
-        <gazebo reference="${side}_rocker">
-            <!-- <material>Gazebo/Blue</material> -->
-            <turnGravityOff>false</turnGravityOff>
-        </gazebo>
-    </xacro:macro>
-    <rocker side="left" parent="chassis" translateX="0" translateY="0" translateZ="0" flipY="1" />
-    <rocker side="right" parent="chassis" translateX="0" translateY="0" translateZ="0" flipY="-1" />
-    <!-- Camera gazebo sensor -->
-    <joint name="camera_joint" type="fixed">
-        <axis xyz="0 1 0" />
-        <origin xyz="${base_lenght / 2 + 2 * camera_size} 0 ${base_height / 2}" rpy="0 0 0"/>
-        <parent link="chassis"/>
-        <child link="camera_link"/>
-    </joint>
-    <link name="camera_link">
-    </link>
-    <link name="camera_link2">
-    </link>
-    <joint name="camera_joint2" type="fixed">
-        <axis xyz="0 1 0" />
-        <origin xyz="0 0 0" rpy="${-M_PI_2} 0 ${-M_PI_2}"/>
-        <parent link="camera_link"/>
-        <child link="camera_link2"/>
-    </joint>
-    <gazebo reference="camera_link">
-        <sensor type="camera" name="camera1">
-            <update_rate>30.0</update_rate>
-            <camera name="head">
-                <horizontal_fov>${45 * DEG_TO_RAD}</horizontal_fov>
-                <image>
-                    <width>2056</width>
-                    <height>1542</height>
-                    <format>R8G8B8</format>
-                </image>
-                <clip>
-                    <near>0.02</near>
-                    <far>300</far>
-                </clip>
-                <noise>
-                    <type>gaussian</type>
-                    <!-- Noise is sampled independently per pixel on each frame.
-               That pixel's noise value is added to each of its color
-               channels, which at that point lie in the range [0,1]. -->
-                    <mean>0.0</mean>
-                    <stddev>0.07</stddev>
-                </noise>
-            </camera>
-            <plugin name="camera_controller" filename="libgazebo_ros_camera.so">
-                <alwaysOn>true</alwaysOn>
-                <updateRate>0.0</updateRate>
-                <cameraName>sensors/camera1</cameraName>
-                <imageTopicName>image_raw</imageTopicName>
-                <cameraInfoTopicName>camera_info</cameraInfoTopicName>
-                <frameName>camera_link2</frameName>
-                <hackBaseline>0.0</hackBaseline>
-                <distortionK1>0.0</distortionK1>
-                <distortionK2>0.0</distortionK2>
-                <distortionK3>0.0</distortionK3>
-                <distortionT1>0.0</distortionT1>
-                <distortionT2>0.0</distortionT2>
-            </plugin>
-        </sensor>
-    </gazebo>
-    <!-- IMU plugin sensor -->
-    <!-- computed by seperate plugin, without gravity -->
-    <gazebo>
-        <plugin name="imu_plugin" filename="libgazebo_ros_imu.so">
-            <alwaysOn>true</alwaysOn>
-            <bodyName>chassis</bodyName>
-            <topicName>sensors/imu_plugin</topicName>
-            <serviceName>imu_service</serviceName>
-            <gaussianNoise>0.0</gaussianNoise>
-            <updateRate>20.0</updateRate>
-        </plugin>
-    </gazebo>
-    <!-- IMU gazebo sensor -->
-    <!-- computed by gazebo, with gravity -->
-    <gazebo reference="chassis">
-        <gravity>true</gravity>
-        <sensor name="imu_sensor" type="imu">
-            <always_on>true</always_on>
-            <update_rate>50</update_rate>
-            <visualize>true</visualize>
-            <topic>__default_topic__</topic>
-            <plugin filename="libgazebo_ros_imu_sensor.so" name="imu_plugin">
-                <topicName>sensors/imu_gazebo</topicName>
-                <bodyName>chassis</bodyName>
-                <updateRateHZ>20.0</updateRateHZ>
-                <gaussianNoise>0.0</gaussianNoise>
-                <xyzOffset>0 0 0</xyzOffset>
-                <rpyOffset>0 0 0</rpyOffset>
-                <frameName>chassis</frameName>
-            </plugin>
-            <pose>0 0 0 0 0 0</pose>
-        </sensor>
-    </gazebo>
+    <!--   rover body macro   -->
+    <body parent="base_link" translateX="0" translateY="0" translateZ="0.1"/>
     <!-- Publishing joint states from Gazebo simulator -->
     <!-- fixed links are not published -->
