Commit message: stereo camera for sim

File: rover_config/urdf/body.xacro (robot description, xacro)
@@ -124,28 +124,29 @@
         <rocker side="right" parent="chassis" translateX="0" translateY="0" translateZ="0" flipY="-1" />
         <!-- Camera gazebo sensor -->
+        <joint name="pre_camera_joint" type="fixed">
+            <axis xyz="0 1 0" />
+            <origin xyz="${base_lenght / 2 + 2 * camera_size} 0 ${base_height / 2}" rpy="0 0.4 0"/>
+            <parent link="chassis"/>
+            <child link="pre_camera_link"/>
+        </joint>
+        <link name="pre_camera_link">
+        </link>
         <joint name="camera_joint" type="fixed">
             <axis xyz="0 1 0" />
-            <origin xyz="${base_lenght / 2 + 2 * camera_size} 0 ${base_height / 2}" rpy="0 0 0"/>
-            <parent link="chassis"/>
+            <origin xyz="0 0 0" rpy="0 0 0"/>
+            <parent link="pre_camera_link"/>
             <child link="camera_link"/>
         </joint>
         <link name="camera_link">
         </link>
-        <link name="camera_link2">
-        </link>
-        <joint name="camera_joint2" type="fixed">
-            <axis xyz="0 1 0" />
-            <origin xyz="0 0 0" rpy="${-M_PI_2} 0 ${-M_PI_2}"/>
-            <parent link="camera_link"/>
-            <child link="camera_link2"/>
-        </joint>
         <gazebo reference="camera_link">
-            <sensor type="camera" name="camera1">
+            <sensor type="multicamera" name="stereo_camera">
                 <update_rate>30.0</update_rate>
-                <camera name="head">
-                    <horizontal_fov>${45 * DEG_TO_RAD}</horizontal_fov>
+                <camera name="left">
+                <pose>0 0.05 0 0 0 0</pose>
+                    <horizontal_fov>${90 * DEG_TO_RAD}</horizontal_fov>
                     <image>
-                        <width>2056</width>
-                        <height>1542</height>
+                        <width>450</width>
+                        <height>300</height>
                         <format>R8G8B8</format>
                     </image>
@@ -154,21 +155,26 @@
                         <far>300</far>
                     </clip>
-                    <noise>
-                        <type>gaussian</type>
-                        <!-- Noise is sampled independently per pixel on each frame.
-                That pixel's noise value is added to each of its color
-                channels, which at that point lie in the range [0,1]. -->
-                        <mean>0.0</mean>
-                        <stddev>0.07</stddev>
-                    </noise>
                 </camera>
-                <plugin name="camera_controller" filename="libgazebo_ros_camera.so">
+                <camera name="right">
+                <pose>0 -0.05 0 0 0 0</pose>
+                    <horizontal_fov>${90 * DEG_TO_RAD}</horizontal_fov>
+                    <image>
+                        <width>450</width>
+                        <height>300</height>
+                        <format>R8G8B8</format>
+                    </image>
+                    <clip>
+                        <near>0.02</near>
+                        <far>300</far>
+                    </clip>
+                </camera>
+                <plugin name="stereo_camera_controller" filename="libgazebo_ros_multicamera.so">
                     <alwaysOn>true</alwaysOn>
                     <updateRate>0.0</updateRate>
-                    <cameraName>sensors/camera1</cameraName>
+                    <cameraName>stereo_camera</cameraName>
                     <imageTopicName>image_raw</imageTopicName>
                     <cameraInfoTopicName>camera_info</cameraInfoTopicName>
-                    <frameName>camera_link2</frameName>
-                    <hackBaseline>0.0</hackBaseline>
+                    <frameName>camera_link</frameName>
+                    <hackBaseline>0.07</hackBaseline>
                     <distortionK1>0.0</distortionK1>
                     <distortionK2>0.0</distortionK2>
@@ -176,5 +182,5 @@
                     <distortionT1>0.0</distortionT1>
                     <distortionT2>0.0</distortionT2>
-                </plugin>
+            </plugin>
             </sensor>
         </gazebo>

Commit message: stereo camera position on tower

File: rover_config/urdf/body.xacro (robot description, xacro)
@@ -126,5 +126,5 @@
         <joint name="pre_camera_joint" type="fixed">
             <axis xyz="0 1 0" />
-            <origin xyz="${base_lenght / 2 + 2 * camera_size} 0 ${base_height / 2}" rpy="0 0.4 0"/>
+            <origin xyz="-0.3 0 0.9" rpy="0 0.4 0"/>
             <parent link="chassis"/>
             <child link="pre_camera_link"/>
